File: ShinyBarnacle/ShinyBarnacle.kicad_pcb (KiCad board)
At the start: 2 copper layers, 82.5 x 35.5 mm, 77 parts, among them J1 USB_B_Mini, J2 Debug, J3 Conn_02x35_JumperluxCardEdge, J4 Conn_02x35_JumperluxCardEdge, SW1 SW_Push, SW2 SW_Push, SW3 SW_Push, SW4 SW_Push, SW5 SW_DIP_x01, SW6 Select Row, SW7 USB BOOT, SW8 SW_Push, U1 NCP1117-3.3_SOT223, U2 W25Q128JVS, U3 RP2040, Y1 ABLS-12.000MHZ-B4-T

Commit message: Finished the Shiny Barnacle
Parts:
- removed BT1: BatteryHolder_Keystone_2468_2xAAA, Battery:BatteryHolder_Keystone_2468_2xAAA
- removed the C4 at (145.8, 135.3)
- removed D10: D_Small, Diode_SMD:D_SOD-123
- removed the D9 at (47.0, 27.9)
- removed R27: 1K, Resistor_SMD:R_0603_1608Metric_Pad0.98x0.95mm_HandSolder
- removed the SW5 at (98.3, 86.6)
- added C16: 0.1uF, Capacitor_SMD:C_0603_1608Metric_Pad1.08x0.95mm_HandSolder, F.Cu at (69.8, 59.7)
- added R20: 10K, Resistor_SMD:R_0603_1608Metric_Pad0.98x0.95mm_HandSolder, F.Cu at (68.6, 59.7)
- added R26: 47K, Resistor_SMD:R_0603_1608Metric_Pad0.98x0.95mm_HandSolder, F.Cu at (67.3, 59.7)
- added SW9: SW_Push, Button_Switch_SMD:SW_Tactile_SPST_NO_Straight_CK_PTS636Sx25SMTRLFS, F.Cu at (59.7, 59.7)
- added TP10: TestPoint, JumperlessFootprints:TestPoint_Pad_D1.0mm, B.Cu at (73.7, 69.8)
- added TP11: TestPoint, JumperlessFootprints:TestPoint_Pad_D1.0mm, B.Cu at (71.1, 69.8)
- added TP12: TestPoint, JumperlessFootprints:TestPoint_Pad_D1.0mm, B.Cu at (68.6, 69.8)
- added TP13: TestPoint, JumperlessFootprints:TestPoint_D0.75mm, B.Cu at (37.8, 85.2)
- added TP14: TestPoint, JumperlessFootprints:TestPoint_D0.75mm, B.Cu at (39.8, 85.2)
- added TP8: TestPoint, JumperlessFootprints:TestPoint_Pad_D1.0mm, B.Cu at (78.7, 69.8)
- added TP9: TestPoint, JumperlessFootprints:TestPoint_Pad_D1.0mm, B.Cu at (76.2, 69.8)
- J2: moved to B.Cu
- R13: renamed from R8; footprint Resistor_SMD:R_0805_2012Metric_Pad1.20x1.40mm_HandSolder -> Resistor_SMD:R_0603_1608Metric_Pad0.98x0.95mm_HandSolder
- R14: renamed from R9; footprint Resistor_SMD:R_0805_2012Metric_Pad1.20x1.40mm_HandSolder -> Resistor_SMD:R_0603_1608Metric_Pad0.98x0.95mm_HandSolder
- R15: renamed from R11; footprint Resistor_SMD:R_0805_2012Metric_Pad1.20x1.40mm_HandSolder -> Resistor_SMD:R_0603_1608Metric_Pad0.98x0.95mm_HandSolder
- R16: renamed from R4; footprint Resistor_SMD:R_0805_2012Metric_Pad1.20x1.40mm_HandSolder -> Resistor_SMD:R_0603_1608Metric_Pad0.98x0.95mm_HandSolder; moved to F.Cu
- R17: renamed from R14; footprint Resistor_SMD:R_0805_2012Metric_Pad1.20x1.40mm_HandSolder -> Resistor_SMD:R_0603_1608Metric_Pad0.98x0.95mm_HandSolder
- R18: renamed from R16; footprint Resistor_SMD:R_0805_2012Metric_Pad1.20x1.40mm_HandSolder -> Resistor_SMD:R_0603_1608Metric_Pad0.98x0.95mm_HandSolder
- R19: renamed from R26; footprint Resistor_SMD:R_0805_2012Metric_Pad1.20x1.40mm_HandSolder -> Resistor_SMD:R_0603_1608Metric_Pad0.98x0.95mm_HandSolder
- R21: renamed from R10; footprint Resistor_SMD:R_0805_2012Metric_Pad1.20x1.40mm_HandSolder -> Resistor_SMD:R_0603_1608Metric_Pad0.98x0.95mm_HandSolder
- R22: renamed from R3; footprint Resistor_SMD:R_0805_2012Metric_Pad1.20x1.40mm_HandSolder -> Resistor_SMD:R_0603_1608Metric_Pad0.98x0.95mm_HandSolder
- R23: renamed from R13; footprint Resistor_SMD:R_0805_2012Metric_Pad1.20x1.40mm_HandSolder -> Resistor_SMD:R_0603_1608Metric_Pad0.98x0.95mm_HandSolder
- R24: renamed from R15; footprint Resistor_SMD:R_0805_2012Metric_Pad1.20x1.40mm_HandSolder -> Resistor_SMD:R_0603_1608Metric_Pad0.98x0.95mm_HandSolder
- R25: footprint Resistor_SMD:R_0805_2012Metric_Pad1.20x1.40mm_HandSolder -> Resistor_SMD:R_0603_1608Metric_Pad0.98x0.95mm_HandSolder
- SW1: renamed from SW7; footprint Button_Switch_SMD:SW_Tactile_SPST_NO_Straight_CK_PTS636Sx25SMTRLFS -> JumperlessFootprints:Tact_Switch_TS24CA
- TP2: renamed from TP5; moved to B.Cu
- TP6: renamed from TP7; moved to B.Cu
- TP7: renamed from TP8; moved to B.Cu
- moved TP7 132.2 mm to (63.5, 69.8)
- moved TP6 128.4 mm to (66.0, 69.8)
- moved R7 124.6 mm to (54.6, 67.9), turned to 180 degrees
- moved R1 124.0 mm to (53.3, 62.9), turned to 90 degrees
- moved R14 123.4 mm to (52.7, 78.7), turned to 90 degrees
- moved R13 123.1 mm to (51.4, 78.7), turned to -90 degrees
- moved R8 122.9 mm to (54.6, 73.0), turned to 180 degrees
- moved R19 115.9 mm to (86.4, 59.7), turned to 90 degrees
- moved R25 114.8 mm to (85.1, 59.7), turned to -90 degrees
- moved C10 112.0 mm to (54.0, 78.7), turned to 90 degrees
- moved R10 107.8 mm to (72.4, 67.9), turned to 180 degrees
- moved TP2 106.3 mm to (88.9, 69.8)
- moved R11 106.2 mm to (72.4, 73.0), turned to 180 degrees
- moved R12 104.6 mm to (72.4, 78.1), turned to 180 degrees
- moved C9 103.4 mm to (62.4, 76.7)
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- renumbered C6 to C1, C13 to C10, C14 to C11, C8 to C12, C15 to C13, C16 to C14, C18 to C15, C7 to C2, C11 to C3, C1 to C4, C12 to C5, C2 to C6, C3 to C7, C5 to C9, D8 to D2, D1 to D3, D2 to D4, D3 to D5, D4 to D6, D5 to D7, D6 to D8, D7 to D9, R5 to R1, R19 to R10, R20 to R11, R23 to R12, R6 to R2, R1 to R3, R2 to R4, R24 to R5, R7 to R6, R12 to R7, R17 to R8, R18 to R9, SW6 to SW3, SW1 to SW4, SW2 to SW5, SW3 to SW6, SW4 to SW7, TP4 to TP1, TP1 to TP3, TP2 to TP4, TP3 to TP5, U2 to U1, U1 to U2
Connections:
- net Button_2 renamed Button_Circuits
- C11 pad 1: Button_1 -> Button_Clear
- C13 pad 1: Button_3 -> Button_Select
- C14 pad 1: Button_4 -> Button_Cancel
- C15 pad 1: Button_5 -> Button_Color
- D2 pad 2: LED_8 -> LED_0
- J3 pad 66: LED_OUT -> LED_DATA_OUT
- J4 pad 66: LED_OUT -> LED_DATA_OUT
- R15 pad 1: Button_1 -> Button_Clear
- R17 pad 1: Button_3 -> Button_Select
- R18 pad 1: Button_4 -> Button_Cancel
- R19 pad 1: Button_5 -> Button_Color
- U3 pad 11: LED_8 -> Button_Net
- U3 pad 12: Button_1 -> Button_Color
- U3 pad 14: Button_3 -> Button_Clear
- U3 pad 15: Button_4 -> Button_Select
- U3 pad 16: Button_5 -> Button_Cancel
- U3 pad 34: unconnected-(U3-GPIO22-Pad34) -> GPIO_22
- U3 pad 35: unconnected-(U3-GPIO23-Pad35) -> GPIO_23
- U3 pad 36: unconnected-(U3-GPIO24-Pad36) -> GPIO_24
- U3 pad 37: LED_DATA_IN -> LED_DATA_OUT
- U3 pad 38: unconnected-(U3-GPIO26_ADC0-Pad38) -> GPIO_26
- U3 pad 39: unconnected-(U3-GPIO27_ADC1-Pad39) -> GPIO_27
Routing:
- net LED_GND: track 0.00 -> 361.5 mm, vias 0 -> 15
- net LED_5V: track 0.00 -> 242.8 mm, vias 0 -> 5
- net LED_DATA_OUT: track 0.00 -> 100.1 mm, vias 0 -> 7
- net Button_Circuits: track 0.00 -> 79.6 mm, vias 0 -> 2
- net LED_DATA_IN: track 0.00 -> 73.6 mm, vias 0 -> 2
- net Button_Clear: track 0.00 -> 69.5 mm, vias 0 -> 2
- net Button_Select: track 0.00 -> 62.3 mm, vias 0 -> 2
- net Button_Color: track 0.00 -> 61.7 mm, vias 0 -> 2
- net /QSPI_SS: track 0.00 -> 60.5 mm, vias 0 -> 3
- net LED_4: track 0.00 -> 56.5 mm, vias 0 -> 2
- net BOTTOM_RAIL_POS: track 0.00 -> 54.4 mm, vias 0 -> 1
- net Button_Cancel: track 0.00 -> 52.9 mm, vias 0 -> 2
- net TOP_RAIL_NEG: track 0.00 -> 51.5 mm, vias 0 -> 2
- net TOP_RAIL_POS: track 0.00 -> 49.4 mm, vias 0 -> 2
- net /QSPI_SD0: track 0.00 -> 48.9 mm, vias 0 -> 2
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- added copper zone on B.Cu, net (none)
- added copper zone on F.Cu, net (none)
Other:
- board text added: "+"
- board text added: "-"
- board text added: "14"
- board text added: "15"
- board text added: "16"
- board text added: "17"
- board text added: "18"
- board text added: "22"
- board text added: "23"
- board text added: "24"
- board text added: "26"
- board text added: "27"
- board text added: "28"
- board text added: "29"
- board text added: "BOOT"
- board text added: "Edit"
- board text added: "GPIO"
- board text added: "Kevin Santo Cappuccio"
- board text added: "Shiny Barnacle"
- board text removed: "Delete"
- board text removed: "Highlight"
- board text removed: "Mode"
