File: ShinyBarnacle/ShinyBarnacle.kicad_sch (KiCad schematic)
At the start: 77 parts, among them J1 USB_B_Mini, J2 Debug, J3 Conn_02x35_JumperluxCardEdge, J4 Conn_02x35_JumperluxCardEdge, SW1 SW_Push, SW2 SW_Push, SW3 SW_Push, SW4 SW_Push, SW5 SW_DIP_x01, SW6 Select Row, SW7 USB BOOT, SW8 SW_Push, U1 NCP1117-3.3_SOT223, U2 W25Q128JVS, U3 RP2040, Y1 ABLS-12.000MHZ-B4-T

Commit message: Finished the Shiny Barnacle
Parts:
- removed BT1: Battery, symbol Device:Battery
- removed C4: 1u, Capacitor_SMD:C_0603_1608Metric_Pad1.08x0.95mm_HandSolder, symbol JumperlessSymbols:C
- removed D10: D_Small, Diode_SMD:D_SOD-123, symbol Device:D_Small
- removed D9: LED, LED_SMD:LED_PLCC-2_3x2mm_AK, symbol Device:LED
- removed R27: 1K, Resistor_SMD:R_0603_1608Metric_Pad0.98x0.95mm_HandSolder, symbol JumperlessSymbols:R_Small_US_3
- removed SW5: SW_DIP_x01, Button_Switch_SMD:SW_DIP_SPSTx01_Slide_6.7x4.1mm_W8.61mm_P2.54mm_LowProfile, symbol Switch:SW_DIP_x01
- added C16: 0.1uF, Capacitor_SMD:C_0603_1608Metric_Pad1.08x0.95mm_HandSolder, symbol JumperlessSymbols:C_Small
- added R20: 10K, Resistor_SMD:R_0603_1608Metric_Pad0.98x0.95mm_HandSolder, symbol JumperlessSymbols:R_Small_US_3
- added R26: 47K, Resistor_SMD:R_0603_1608Metric_Pad0.98x0.95mm_HandSolder, symbol JumperlessSymbols:R_Small_US_3
- added SW9: SW_Push, Button_Switch_SMD:SW_Tactile_SPST_NO_Straight_CK_PTS636Sx25SMTRLFS, symbol JumperlessSymbols:SW_Push
- added TP10, TP11, TP12, TP13, TP14, TP8, TP9: TestPoint, JumperlessFootprints:TestPoint_Pad_D1.0mm, symbol Connector:TestPoint
- R13: renamed from R8; footprint Resistor_SMD:R_0805_2012Metric_Pad1.20x1.40mm_HandSolder -> Resistor_SMD:R_0603_1608Metric_Pad0.98x0.95mm_HandSolder
- R14: renamed from R9; footprint Resistor_SMD:R_0805_2012Metric_Pad1.20x1.40mm_HandSolder -> Resistor_SMD:R_0603_1608Metric_Pad0.98x0.95mm_HandSolder
- R15: renamed from R11; footprint Resistor_SMD:R_0805_2012Metric_Pad1.20x1.40mm_HandSolder -> Resistor_SMD:R_0603_1608Metric_Pad0.98x0.95mm_HandSolder
- R16: renamed from R4; footprint Resistor_SMD:R_0805_2012Metric_Pad1.20x1.40mm_HandSolder -> Resistor_SMD:R_0603_1608Metric_Pad0.98x0.95mm_HandSolder
- R17: renamed from R14; footprint Resistor_SMD:R_0805_2012Metric_Pad1.20x1.40mm_HandSolder -> Resistor_SMD:R_0603_1608Metric_Pad0.98x0.95mm_HandSolder
- R18: renamed from R16; footprint Resistor_SMD:R_0805_2012Metric_Pad1.20x1.40mm_HandSolder -> Resistor_SMD:R_0603_1608Metric_Pad0.98x0.95mm_HandSolder
- R19: renamed from R26; footprint Resistor_SMD:R_0805_2012Metric_Pad1.20x1.40mm_HandSolder -> Resistor_SMD:R_0603_1608Metric_Pad0.98x0.95mm_HandSolder
- R21: renamed from R10; footprint Resistor_SMD:R_0805_2012Metric_Pad1.20x1.40mm_HandSolder -> Resistor_SMD:R_0603_1608Metric_Pad0.98x0.95mm_HandSolder
- R22: renamed from R3; footprint Resistor_SMD:R_0805_2012Metric_Pad1.20x1.40mm_HandSolder -> Resistor_SMD:R_0603_1608Metric_Pad0.98x0.95mm_HandSolder
- R23: renamed from R13; footprint Resistor_SMD:R_0805_2012Metric_Pad1.20x1.40mm_HandSolder -> Resistor_SMD:R_0603_1608Metric_Pad0.98x0.95mm_HandSolder
- R24: renamed from R15; footprint Resistor_SMD:R_0805_2012Metric_Pad1.20x1.40mm_HandSolder -> Resistor_SMD:R_0603_1608Metric_Pad0.98x0.95mm_HandSolder
- R25: footprint Resistor_SMD:R_0805_2012Metric_Pad1.20x1.40mm_HandSolder -> Resistor_SMD:R_0603_1608Metric_Pad0.98x0.95mm_HandSolder
- SW1: renamed from SW7; footprint Button_Switch_SMD:SW_Tactile_SPST_NO_Straight_CK_PTS636Sx25SMTRLFS -> JumperlessFootprints:Tact_Switch_TS24CA
- renumbered C6 to C1, C13 to C10, C14 to C11, C8 to C12, C15 to C13, C16 to C14, C18 to C15, C7 to C2, C11 to C3, C1 to C4, C12 to C5, C2 to C6, C3 to C7, C5 to C9, D8 to D2, D1 to D3, D2 to D4, D3 to D5, D4 to D6, D5 to D7, D6 to D8, D7 to D9, R5 to R1, R19 to R10, R20 to R11, R23 to R12, R6 to R2, R1 to R3, R2 to R4, R24 to R5, R7 to R6, R12 to R7, R17 to R8, R18 to R9, SW6 to SW3, SW1 to SW4, SW2 to SW5, SW3 to SW6, SW4 to SW7, TP4 to TP1, TP5 to TP2, TP1 to TP3, TP2 to TP4, TP3 to TP5, TP7 to TP6, TP8 to TP7, U2 to U1, U1 to U2
Connections:
- net +3V3: now also R26.2
- net GND: now also C16.2, SW9.1
- net LED_0: now also D2.2 (A)
- net LED_DATA_IN: now also TP13.1; no longer U3.37 (GPIO25)
- net GPIO_22: now reaches U3.34 (GPIO22)
- net GPIO_22: now also TP8.1
- net GPIO_23: now reaches U3.35 (GPIO23)
- net GPIO_23: now also TP9.1
- net GPIO_24: now reaches U3.36 (GPIO24)
- net GPIO_24: now also TP10.1
- net GPIO_26: now reaches U3.38 (GPIO26_ADC0)
- net GPIO_26: now also TP11.1
- net GPIO_27: now reaches U3.39 (GPIO27_ADC1)
- net GPIO_27: now also TP12.1
- net Button_1 renamed Button_Clear
- net Button_Clear: now also U3.14 (GPIO11); no longer U3.12 (GPIO9)
- net Button_2 renamed Button_Circuits
- net Button_3 renamed Button_Select
- net Button_Select: now also U3.15 (GPIO12); no longer U3.14 (GPIO11)
- net Button_4 renamed Button_Cancel
- net Button_Cancel: now also U3.16 (GPIO13); no longer U3.15 (GPIO12)
- net Button_5 renamed Button_Color
- net Button_Color: now also U3.12 (GPIO9); no longer U3.16 (GPIO13)
- net LED_8 renamed Button_Net
- net Button_Net: now also C16.1, R20.1; no longer D2.2 (A)
- net LED_OUT renamed LED_DATA_OUT
- net LED_DATA_OUT: now also U3.37 (GPIO25), TP14.1
- new net: R20.2, R26.1, SW9.2
Other:
- moved on the sheet: D2, D3, D4, D5, D6, D7, D8, D9, R10, R11, R12, R5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
