File: BarnacleBoard/BarnacleBoard.kicad_pcb (KiCad board)
At the start: 2 copper layers, 82.6 x 63.4 mm, 114 parts, among them J1 Conn_02x35_Top_Bottom, J11 Connector_Breadboard, J12 Conn_02x03_Top_Bottom, J13 Conn_02x03_Top_Bottom, J14 Conn_01x06, J15 Conn_01x01, J2 pad_sense_1, J3 pad_sense_30, J4 pad_sense_60, J5 pad_sense_31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

Commit message: actually route most of the barnacles
Parts:
- J11: footprint JumperlessFootprints:Breadboard_CustomClips_CorrectPins_1 -> JumperlessFootprints:Breadboard_CustomClips_CorrectPins_2
