File: BarnacleBoard/BarnacleBoard.kicad_sch (KiCad schematic)
At the start: 41 parts, among them J1 Conn_02x35_Top_Bottom, J10 Conn_01x03, J11 Connector_Breadboard, J12 Conn_02x03_Top_Bottom, J13 Conn_02x03_Top_Bottom, J14 Conn_01x06, J15 Conn_01x01, J2 pad_sense_1, J3 pad_sense_30, J4 pad_sense_60, J5 pad_sense_31, J6 Conn_02x35_Top_Bottom, J7 Conn_01x03, J8 J8, J9 RIGHT

Commit message: add wigs
Parts:
- added J16: Conn_02x35_Top_Bottom, WaferSpace:CONN-SMD_70P-P0.40_HCTL_HC-PBB40C-70DP-0.4V-02, symbol Connector_Generic:Conn_02x35_JumperluxCardEdge
Connections:
- net +5V: now also J16.70 (Pin_70)
- net GND: now also J16.68 (Pin_68)
- net LED_IN: no longer J1.69 (Pin_69), J14.1 (Pin_1), J14.2 (Pin_2), J6.69 (Pin_69), J7.2 (Pin_2), TP16.1, TP17.1
- net PASS: now reaches J1.65 (Pin_65), J15.1 (Pin_1), J6.65 (Pin_65)
- net PASS: now also J16.65 (Pin_65)
- net 1: now reaches J1.1 (Pin_1), J11.1 (Pin_1), J6.1 (Pin_1)
- net 1: now also J16.1 (Pin_1)
- net 10: now reaches J1.10 (Pin_10), J11.10 (Pin_10), J6.10 (Pin_10)
- net 10: now also J16.10 (Pin_10)
- net 11: now reaches J1.11 (Pin_11), J11.11 (Pin_11), J6.11 (Pin_11)
- net 11: now also J16.11 (Pin_11)
- net 12: now reaches J1.12 (Pin_12), J11.12 (Pin_12), J6.12 (Pin_12)
- net 12: now also J16.12 (Pin_12)
- net 13: now reaches J1.13 (Pin_13), J11.13 (Pin_13), J6.13 (Pin_13)
- net 13: now also J16.13 (Pin_13)
- net 14: now reaches J1.14 (Pin_14), J11.14 (Pin_14), J6.14 (Pin_14)
- net 14: now also J16.14 (Pin_14)
- net 15: now reaches J1.15 (Pin_15), J11.15 (Pin_15), J6.15 (Pin_15)
- net 15: now also J16.15 (Pin_15)
- net 16: now reaches J1.16 (Pin_16), J11.16 (Pin_16), J6.16 (Pin_16)
- net 16: now also J16.16 (Pin_16)
- net 17: now reaches J1.17 (Pin_17), J11.17 (Pin_17), J6.17 (Pin_17)
- net 17: now also J16.17 (Pin_17)
- net 18: now reaches J1.18 (Pin_18), J11.18 (Pin_18), J6.18 (Pin_18)
- net 18: now also J16.18 (Pin_18)
- net 19: now reaches J1.19 (Pin_19), J11.19 (Pin_19), J6.19 (Pin_19)
- net 19: now also J16.19 (Pin_19)
- net 2: now reaches J1.2 (Pin_2), J11.2 (Pin_2), J6.2 (Pin_2)
- net 2: now also J16.2 (Pin_2)
- net 20: now reaches J1.20 (Pin_20), J11.20 (Pin_20), J6.20 (Pin_20)
- net 20: now also J16.20 (Pin_20)
- net 21: now reaches J1.21 (Pin_21), J11.21 (Pin_21), J6.21 (Pin_21)
- net 21: now also J16.21 (Pin_21)
- net 22: now reaches J1.22 (Pin_22), J11.22 (Pin_22), J6.22 (Pin_22)
- net 22: now also J16.22 (Pin_22)
- net 23: now reaches J1.23 (Pin_23), J11.23 (Pin_23), J6.23 (Pin_23)
- net 23: now also J16.23 (Pin_23)
- net 24: now reaches J1.24 (Pin_24), J11.24 (Pin_24), J6.24 (Pin_24)
- net 24: now also J16.24 (Pin_24)
- net 25: now reaches J1.25 (Pin_25), J11.25 (Pin_25), J6.25 (Pin_25)
- net 25: now also J16.25 (Pin_25)
- net 26: now reaches J1.26 (Pin_26), J11.26 (Pin_26), J6.26 (Pin_26)
- net 26: now also J16.26 (Pin_26)
- net 27: now reaches J1.27 (Pin_27), J11.27 (Pin_27), J6.27 (Pin_27)
- net 27: now also J16.27 (Pin_27)
- net 28: now reaches J1.28 (Pin_28), J11.28 (Pin_28), J6.28 (Pin_28)
- net 28: now also J16.28 (Pin_28)
- net 29: now reaches J1.29 (Pin_29), J11.29 (Pin_29), J6.29 (Pin_29)
- net 29: now also J16.29 (Pin_29)
- net 3: now reaches J1.3 (Pin_3), J11.3 (Pin_3), J6.3 (Pin_3)
- net 3: now also J16.3 (Pin_3)
- net 30: now reaches J1.30 (Pin_30), J11.30 (Pin_30), J6.30 (Pin_30)
- net 30: now also J16.30 (Pin_30)
- net 31: now reaches J1.31 (Pin_31), J11.31 (Pin_31), J6.31 (Pin_31)
- net 31: now also J16.31 (Pin_31)
- net 32: now reaches J1.32 (Pin_32), J11.32 (Pin_0), J6.32 (Pin_32)
- net 32: now also J16.32 (Pin_32)
- net 33: now reaches J1.33 (Pin_33), J11.33 (Pin_1), J6.33 (Pin_33)
- net 33: now also J16.33 (Pin_33)
- net 34: now reaches J1.34 (Pin_34), J11.34 (Pin_2), J6.34 (Pin_34)
- net 34: now also J16.34 (Pin_34)
- net 35: now reaches J1.35 (Pin_35), J11.35 (Pin_3), J6.35 (Pin_35)
- net 35: now also J16.35 (Pin_35)
- net 36: now reaches J1.36 (Pin_36), J11.36 (Pin_4), J6.36 (Pin_36)
- net 36: now also J16.36 (Pin_36)
- net 37: now reaches J1.37 (Pin_37), J11.37 (Pin_5), J6.37 (Pin_37)
- net 37: now also J16.37 (Pin_37)
- net 38: now reaches J1.38 (Pin_38), J11.38 (Pin_6), J6.38 (Pin_38)
- net 38: now also J16.38 (Pin_38)
- net 39: now reaches J1.39 (Pin_39), J11.39 (Pin_7), J6.39 (Pin_39)
- net 39: now also J16.39 (Pin_39)
- net 4: now reaches J1.4 (Pin_4), J11.4 (Pin_4), J6.4 (Pin_4)
- net 4: now also J16.4 (Pin_4)
- net 40: now reaches J1.40 (Pin_40), J11.40 (Pin_8), J6.40 (Pin_40)
- net 40: now also J16.40 (Pin_40)
- net 41: now reaches J1.41 (Pin_41), J11.41 (Pin_9), J6.41 (Pin_41)
- net 41: now also J16.41 (Pin_41)
- net 42: now reaches J1.42 (Pin_42), J11.42 (Pin_10), J6.42 (Pin_42)
- net 42: now also J16.42 (Pin_42)
- net 43: now reaches J1.43 (Pin_43), J11.43 (Pin_11), J6.43 (Pin_43)
- net 43: now also J16.43 (Pin_43)
- net 44: now reaches J1.44 (Pin_44), J11.44 (Pin_12), J6.44 (Pin_44)
- net 44: now also J16.44 (Pin_44)
- net 45: now reaches J1.45 (Pin_45), J11.45 (Pin_13), J6.45 (Pin_45)
- net 45: now also J16.45 (Pin_45)
- net 46: now reaches J1.46 (Pin_46), J11.46 (Pin_14), J6.46 (Pin_46)
- net 46: now also J16.46 (Pin_46)
- net 47: now reaches J1.47 (Pin_47), J11.47 (Pin_15), J6.47 (Pin_47)
- net 47: now also J16.47 (Pin_47)
- net 48: now reaches J1.48 (Pin_48), J11.48 (Pin_16), J6.48 (Pin_48)
- net 48: now also J16.48 (Pin_48)
- net 49: now reaches J1.49 (Pin_49), J11.49 (Pin_17), J6.49 (Pin_49)
- net 49: now also J16.49 (Pin_49)
- net 5: now reaches J1.5 (Pin_5), J11.5 (Pin_5), J6.5 (Pin_5)
- net 5: now also J16.5 (Pin_5)
- net 50: now reaches J1.50 (Pin_50), J11.50 (Pin_18), J6.50 (Pin_50)
- net 50: now also J16.50 (Pin_50)
- net 51: now reaches J1.51 (Pin_51), J11.51 (Pin_19), J6.51 (Pin_51)
- net 51: now also J16.51 (Pin_51)
- net 52: now reaches J1.52 (Pin_52), J11.52 (Pin_20), J6.52 (Pin_52)
- net 52: now also J16.52 (Pin_52)
- net 53: now reaches J1.53 (Pin_53), J11.53 (Pin_21), J6.53 (Pin_53)
- net 53: now also J16.53 (Pin_53)
- net 54: now reaches J1.54 (Pin_54), J11.54 (Pin_22), J6.54 (Pin_54)
- net 54: now also J16.54 (Pin_54)
- net 55: now reaches J1.55 (Pin_55), J11.55 (Pin_23), J6.55 (Pin_55)
- net 55: now also J16.55 (Pin_55)
- net 56: now reaches J1.56 (Pin_56), J11.56 (Pin_24), J6.56 (Pin_56)
- net 56: now also J16.56 (Pin_56)
- net 57: now reaches J1.57 (Pin_57), J11.57 (Pin_25), J6.57 (Pin_57)
- net 57: now also J16.57 (Pin_57)
- net 58: now reaches J1.58 (Pin_58), J11.58 (Pin_26), J6.58 (Pin_58)
- net 58: now also J16.58 (Pin_58)
- net 59: now reaches J1.59 (Pin_59), J11.59 (Pin_27), J6.59 (Pin_59)
- net 59: now also J16.59 (Pin_59)
- net 6: now reaches J1.6 (Pin_6), J11.6 (Pin_6), J6.6 (Pin_6)
- net 6: now also J16.6 (Pin_6)
- net 60: now reaches J1.60 (Pin_60), J11.60 (Pin_28), J6.60 (Pin_60)
- net 60: now also J16.60 (Pin_60)
- net 7: now reaches J1.7 (Pin_7), J11.7 (Pin_7), J6.7 (Pin_7)
- net 7: now also J16.7 (Pin_7)
- net 8: now reaches J1.8 (Pin_8), J11.8 (Pin_8), J6.8 (Pin_8)
- net 8: now also J16.8 (Pin_8)
- net 9: now reaches J1.9 (Pin_9), J11.9 (Pin_9), J6.9 (Pin_9)
- net 9: now also J16.9 (Pin_9)
- net BOT_NEG renamed BOT_RAIL_NEG
- net BOT_RAIL_NEG: now also J16.64 (Pin_64)
- net BOT_POS renamed BOT_RAIL_POS
- net BOT_RAIL_POS: now also J16.63 (Pin_63)
- net PAD_SENSE_IN renamed SENSE_TOP
- net SENSE_TOP: now also J16.66 (Pin_66)
- net PAD_SENSE_OUT renamed SENSE_BOTTOM
- net SENSE_BOTTOM: now also J16.67 (Pin_67)
- net TOP_NEG renamed TOP_RAIL_NEG
- net TOP_RAIL_NEG: now also J16.62 (Pin_62)
- net TOP_POS renamed TOP_RAIL_POS
- net TOP_RAIL_POS: now also J16.61 (Pin_61)
- new net LED_DAT: J1.69 (Pin_69), J14.1 (Pin_1), J14.2 (Pin_2), J16.69 (Pin_69), J6.69 (Pin_69), J7.2 (Pin_2), TP16.1, TP17.1
Other:
- moved on the sheet: J1, J11A, J6, TP18, TP21, TP22
