File: Barnacles/SMD/SMD.kicad_pcb (KiCad board)
At the start: 4 copper layers, 82.6 x 17.3 mm, 36 parts, among them J1 Conn_01x01, J1 Conn_02x35_Top_Bottom, J12 Conn_02x03_Top_Bottom, J12 Conn_02x32_Top_Bottom, J13 Conn_02x03_Top_Bottom, J13 Conn_02x32_Top_Bottom, J14 Conn_02x32_Top_Bottom, J15 Conn_02x30_Top_Bottom, J16 Conn_02x32_Top_Bottom, J17 Conn_01x30_Socket, J18 Conn_01x30_Socket, J2 Conn_01x01, J3 Conn_01x01, J4 Conn_01x01, J5 Conn_01x01, J6 Conn_02x35_Top_Bottom

Commit message: finish SMD barnacle
Parts:
- removed the J1 at (11.6, 66.3)
- removed the J2 at (13.1, 66.3)
- removed the J3 at (-28.8, 66.3)
- removed the J4 at (-30.3, 66.3)
- removed the J5 at (-8.61, 66.3)
- removed the REF** at (-49.9, 62.1)
- removed the REF** at (32.7, 62.1)
- removed TP17: LED DIN, Connector_PinHeader_2.54mm:PinHeader_1x01_P2.54mm_Vertical_Rounded
- removed TP18: LED 5V, Connector_PinHeader_2.54mm:PinHeader_1x01_P2.54mm_Vertical_Rounded
- removed TP19: LED GND, Connector_PinHeader_2.54mm:PinHeader_1x01_P2.54mm_Vertical_Rounded
- removed the U1 at (16.8, 73.5)
- removed U2: ~, JumperlessFootprints:Conn_2x30_breadboard_double
- removed U2: ~, JumperlessFootprints:Conn_8x30_breadboard
- removed the U3 at (21.9, 48.6)
- added ?: , , F.Cu at (168.5, 49.6)
- added ?: , , F.Cu at (242.2, 57.9)
- added ?: , , F.Cu at (227.0, 42.7)
- added ?: , , F.Cu at (176.2, 59.8)
- added ?: , , F.Cu at (170.5, 47.7)
- added ?: , , F.Cu at (221.9, 46.5)
- added ?: , , F.Cu at (242.2, 40.8)
- added ?: , , F.Cu at (176.2, 40.8)
- added ?: , , F.Cu at (227.0, 56.0)
- added ?: , , F.Cu at (216.8, 61.7)
- added ?: , , F.Cu at (216.8, 40.8)
- added ?: , , F.Cu at (166.6, 61.1)
- added ? (x2): , , F.Cu at (242.2, 42.7)
- added ?: , , F.Cu at (198.4, 61.7)
- added ?: , , F.Cu at (190.1, 44.6)
- added ?: , , F.Cu at (221.9, 42.7)
- added ?: , , F.Cu at (219.3, 44.6)
- added ?: , , F.Cu at (242.2, 48.4)
- added ?: , , F.Cu at (239.7, 61.7)
- added ?: , , F.Cu at (168.5, 47.7)
- added ?: , , F.Cu at (178.7, 40.8)
- added ?: , , F.Cu at (229.5, 48.4)
- added ?: , , F.Cu at (170.5, 49.6)
- added ?: , , F.Cu at (192.0, 44.6)
- added ?: , , F.Cu at (166.6, 51.5)
- added ?: , , F.Cu at (168.5, 51.5)
- added ?: , , F.Cu at (239.7, 46.5)
- added ?: , , F.Cu at (224.4, 48.4)
- added ?: , , F.Cu at (193.9, 44.6)
- added ?: , , F.Cu at (242.2, 54.1)
- added ?: , , F.Cu at (232.0, 56.0)
- added ?: , , F.Cu at (181.2, 45.8)
- added ?: , , F.Cu at (221.9, 40.8)
- added ?: , , F.Cu at (209.2, 40.8)
- added ?: , , F.Cu at (168.5, 55.4)
- added ?: , , F.Cu at (209.2, 61.7)
- added ?: , , F.Cu at (214.3, 56.0)
- added ?: , , F.Cu at (214.3, 44.6)
- added ?: , , F.Cu at (204.1, 40.8)
- added ?: , , F.Cu at (204.1, 61.7)
- added ?: , , F.Cu at (239.7, 54.1)
- added ?: , , F.Cu at (166.6, 49.6)
- added ?: , , F.Cu at (237.1, 46.5)
- added ?: , , F.Cu at (166.6, 45.8)
- added ?: , , F.Cu at (219.3, 46.5)
- added ?: , , F.Cu at (242.2, 46.5)
- added ?: , , F.Cu at (201.6, 42.7)
- added ?: , , F.Cu at (198.4, 59.8)
- added ?: , , F.Cu at (239.7, 42.7)
- added ?: , , F.Cu at (237.1, 48.4)
- added ?: , , F.Cu at (206.6, 61.7)
- added ?: , , F.Cu at (166.6, 55.4)
- added ?: , , F.Cu at (202.2, 61.7)
- added ?: , , F.Cu at (178.7, 61.7)
- added ?: , , F.Cu at (211.7, 40.8)
- added ?: , , F.Cu at (219.3, 56.0)
- added ?: , , F.Cu at (199.7, 44.6)
- added ?: , , F.Cu at (181.2, 56.6)
- added ?: , , F.Cu at (224.4, 54.1)
- added ?: , , F.Cu at (171.1, 61.7)
- added ?: , , F.Cu at (168.5, 57.3)
- added ?: , , F.Cu at (232.0, 54.1)
- added ?: , , F.Cu at (242.2, 50.3)
- added ?: , , F.Cu at (166.6, 59.2)
- added ?: , , F.Cu at (224.4, 56.0)
- added ?: , , F.Cu at (219.3, 57.9)
- added ?: , , F.Cu at (204.1, 59.8)
- added ?: , , F.Cu at (242.2, 61.7)
- added ?: , , F.Cu at (166.6, 57.3)
- added ?: , , F.Cu at (234.6, 54.1)
- added ?: , , F.Cu at (227.0, 54.1)
- added ?: , , F.Cu at (196.5, 40.8)
- added ?: , , F.Cu at (194.0, 40.7)
- added ?: , , F.Cu at (168.5, 59.2)
- added ?: , , F.Cu at (237.1, 54.1)
- added ?: , , F.Cu at (234.6, 42.7)
- added ?: , , F.Cu at (172.4, 55.4)
- added ?: , , F.Cu at (234.6, 48.4)
- added ?: , , F.Cu at (214.3, 61.7)
- added ?: , , F.Cu at (206.6, 40.8)
- added ?: , , F.Cu at (242.2, 44.6)
- added ? (x2): , , F.Cu at (242.2, 59.8)
- added ?: , , F.Cu at (176.2, 61.7)
- added ?: , , F.Cu at (166.6, 43.9)
- added ?: , , F.Cu at (198.4, 57.9)
- added ?: , , F.Cu at (219.3, 61.7)
- added ?: , , F.Cu at (204.1, 42.7)
- added ?: , , F.Cu at (227.0, 46.5)
- added ?: , , F.Cu at (211.7, 56.0)
- added ?: , , F.Cu at (206.6, 42.7)
- added ?: , , F.Cu at (237.1, 40.8)
- added ?: , , F.Cu at (173.6, 40.8)
- added ?: , , F.Cu at (239.7, 50.3)
- added ?: , , F.Cu at (237.1, 56.0)
- added ?: , , F.Cu at (211.7, 46.5)
- added ?: , , F.Cu at (168.5, 53.5)
- added ?: , , F.Cu at (176.2, 42.7)
- added ?: , , F.Cu at (166.6, 42.0)
- added ?: , , F.Cu at (197.8, 44.6)
- added ?: , , F.Cu at (224.4, 40.8)
- added ?: , , F.Cu at (232.0, 42.7)
- added ?: , , F.Cu at (229.5, 56.0)
- added ?: , , F.Cu at (229.5, 46.5)
- added ?: , , F.Cu at (224.4, 46.5)
- added ?: , , F.Cu at (166.6, 47.7)
- added ?: , , F.Cu at (214.3, 46.5)
- added ?: , , F.Cu at (234.6, 46.5)
- added ?: , , F.Cu at (192.7, 57.9)
- added ?: , , F.Cu at (216.8, 46.5)
- added ?: , , F.Cu at (211.7, 57.9)
- added ?: , , F.Cu at (195.9, 44.6)
- added ?: , , F.Cu at (234.6, 40.8)
- added ?: , , F.Cu at (173.6, 42.7)
- added ?: , , F.Cu at (242.2, 56.0)
- added ?: , , F.Cu at (173.6, 61.7)
- added ?: , , F.Cu at (229.5, 42.7)
- added ?: , , F.Cu at (166.6, 53.5)
- added ?: , , F.Cu at (173.6, 59.8)
- added ?: , , F.Cu at (239.7, 48.4)
- added ?: , , F.Cu at (202.2, 59.8)
- added ?: , , F.Cu at (242.2, 52.2)
- added ?: , , F.Cu at (214.3, 57.9)
- added ?: , , F.Cu at (214.3, 40.8)
- added ?: , , F.Cu at (211.7, 44.6)
- added ?: , , F.Cu at (196.5, 57.9)
- added ?: , , F.Cu at (199.7, 42.7)
- added ?: , , F.Cu at (232.0, 46.5)
- added ?: , , F.Cu at (194.6, 57.9)
- added ?: , , F.Cu at (190.8, 57.9)
- added ?: , , F.Cu at (224.4, 42.7)
- added ?: , , F.Cu at (229.5, 40.8)
- added ?: , , F.Cu at (232.0, 48.4)
- added ?: , , F.Cu at (227.0, 40.8)
- added ?: , , F.Cu at (229.5, 54.1)
- added ?: , , F.Cu at (216.8, 44.6)
- added ?: , , F.Cu at (196.5, 59.8)
- added ?: , , F.Cu at (170.5, 45.8)
- added ?: , , F.Cu at (234.6, 56.0)
- added ?: , , F.Cu at (200.3, 61.7)
- added ?: , , F.Cu at (201.6, 40.8)
- added ?: , , F.Cu at (206.6, 59.8)
- added ?: , , F.Cu at (219.3, 59.8)
- added ?: , , F.Cu at (216.8, 56.0)
- added ?: , , F.Cu at (170.5, 55.4)
- added ?: , , F.Cu at (232.0, 40.8)
- added ?: , , F.Cu at (183.2, 56.6)
- added ?: , , F.Cu at (209.2, 57.9)
- added ?: , , F.Cu at (239.7, 52.2)
- added ?: , , F.Cu at (239.7, 40.8)
- added ?: , , F.Cu at (170.5, 53.5)
- added ?: , , F.Cu at (211.7, 42.7)
- added ?: , , F.Cu at (170.5, 57.3)
- added ?: , , F.Cu at (183.2, 45.8)
- added ?: , , F.Cu at (200.3, 59.8)
- added ?: , , F.Cu at (170.5, 51.5)
- added ?: , , F.Cu at (219.3, 42.7)
- added ?: , , F.Cu at (237.1, 42.7)
- added ?: , , F.Cu at (239.7, 59.8)
- added ?: , , F.Cu at (219.3, 40.8)
- added ?: , , F.Cu at (172.4, 47.7)
- added ?: , , F.Cu at (171.1, 40.8)
- added ?: , , F.Cu at (239.7, 56.0)
- added ?: , , F.Cu at (227.0, 48.4)
- added ?: , , F.Cu at (168.5, 45.8)
- J1, J6: value Conn_02x35_Top_Bottom -> Conn_01x01
- J12, J13: value Conn_02x03_Top_Bottom -> Conn_02x32_Top_Bottom
- J17, J18: value Conn_01x30_Socket -> Conn_01x30; footprint Connector_PinHeader_2.54mm:PINHEADER_1x30_lemons_unlemoned -> JumperlessFootprints:Conn_1x30_breadboard_single
- moved J17 86.3 mm to (204.1, 66.1), turned to 0 degrees
- moved J12 60.2 mm to (184.1, 51.2)
- moved J13 60.2 mm to (212.5, 51.2)
- moved J14 60.2 mm to (173.6, 51.2)
- moved J15 60.2 mm to (230.3, 51.2)
- moved J16 60.2 mm to (196.8, 51.2)
- moved J18 35.8 mm to (204.1, 36.9), turned to 0 degrees
- moved U3 22.9 mm to (234.6, 30.6)
- moved REF** 21.6 mm to (245.4, 66.5)
- moved REF** 21.6 mm to (162.9, 66.5)
- moved J1 20.9 mm to (224.3, 73.6)
- moved J2 20.9 mm to (225.8, 73.6)
- moved J3 20.9 mm to (183.9, 73.6)
- moved J4 20.9 mm to (182.4, 73.6)
- moved J5 20.9 mm to (204.1, 73.6)
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Connections:
- net Net-(J2-Pin_1) renamed TOP_RAIL_NEG
- net Net-(J3-Pin_1) renamed BOT_RAIL_POS
- net Net-(J4-Pin_1) renamed BOT_RAIL_NEG
- net Net-(J5-Pin_1) renamed PASS
- net Net-(J6-Pin_1) renamed SENSE_TOP
- net Net-(J7-Pin_1) renamed SENSE_BOTTOM
- net Net-(J9-Pin_1) renamed LED_DAT
- J1 pad 1: Net-(J1-Pin_1) -> TOP_RAIL_POS
- J12 pad 1: Net-(J1-Pin_1) -> 31
- J12 pad 10: Net-(J1-Pin_10) -> 40
- J12 pad 11: Net-(J1-Pin_11) -> 41
- J12 pad 12: Net-(J1-Pin_12) -> 42
- J12 pad 13: Net-(J1-Pin_13) -> 43
- J12 pad 14: Net-(J1-Pin_14) -> 44
- J12 pad 15: Net-(J1-Pin_16) -> 46
- J12 pad 16: Net-(J1-Pin_17) -> 47
- J12 pad 17: Net-(J1-Pin_18) -> 48
- J12 pad 18: Net-(J1-Pin_19) -> 49
- J12 pad 19: Net-(J1-Pin_20) -> 50
- J12 pad 2: Net-(J1-Pin_2) -> 32
- J12 pad 20: Net-(J1-Pin_21) -> 51
- J12 pad 21: Net-(J1-Pin_22) -> 52
- J12 pad 22: Net-(J1-Pin_23) -> 53
- J12 pad 23: Net-(J1-Pin_24) -> 54
- J12 pad 24: Net-(J1-Pin_25) -> 55
- J12 pad 25: Net-(J1-Pin_26) -> 56
- J12 pad 26: Net-(J1-Pin_27) -> 57
- J12 pad 27: Net-(J1-Pin_28) -> 58
- J12 pad 28: Net-(J1-Pin_29) -> 59
- J12 pad 29: Net-(J10-Pin_2) -> 29
- J12 pad 3: Net-(J1-Pin_3) -> 33
- J12 pad 30: Net-(J10-Pin_3) -> 28
- J12 pad 31: Net-(J10-Pin_4) -> 27
- J12 pad 32: Net-(J10-Pin_5) -> 26
- J12 pad 33: Net-(J10-Pin_6) -> 25
- J12 pad 34: Net-(J10-Pin_7) -> 24
- J12 pad 35: Net-(J10-Pin_8) -> 23
- J12 pad 36: Net-(J10-Pin_9) -> 22
- J12 pad 37: Net-(J10-Pin_10) -> 21
- J12 pad 38: Net-(J10-Pin_11) -> 20
- J12 pad 39: Net-(J10-Pin_12) -> 19
- J12 pad 4: Net-(J1-Pin_4) -> 34
- J12 pad 40: Net-(J10-Pin_13) -> 18
- J12 pad 41: Net-(J10-Pin_14) -> 17
- J12 pad 42: Net-(J10-Pin_15) -> 16
- J12 pad 43: Net-(J10-Pin_17) -> 14
- J12 pad 44: Net-(J10-Pin_18) -> 13
- J12 pad 45: Net-(J10-Pin_19) -> 12
- J12 pad 46: Net-(J10-Pin_20) -> 11
- J12 pad 47: Net-(J10-Pin_21) -> 10
- J12 pad 48: Net-(J10-Pin_22) -> 9
- J12 pad 49: Net-(J10-Pin_23) -> 8
- J12 pad 5: Net-(J1-Pin_5) -> 35
- J12 pad 50: Net-(J10-Pin_24) -> 7
- J12 pad 51: Net-(J10-Pin_25) -> 6
- J12 pad 52: Net-(J10-Pin_26) -> 5
- J12 pad 53: Net-(J10-Pin_27) -> 4
- J12 pad 54: Net-(J10-Pin_28) -> 3
- J12 pad 55: Net-(J10-Pin_29) -> 2
- J12 pad 56: Net-(J10-Pin_30) -> 1
- J12 pad 6: Net-(J1-Pin_6) -> 36
- J12 pad 7: Net-(J1-Pin_7) -> 37
- J12 pad 8: Net-(J1-Pin_8) -> 38
- J12 pad 9: Net-(J1-Pin_9) -> 39
- J13 pad 1: Net-(J1-Pin_1) -> 31
- J13 pad 10: Net-(J1-Pin_10) -> 40
- J13 pad 11: Net-(J1-Pin_11) -> 41
- J13 pad 12: Net-(J1-Pin_12) -> 42
- J13 pad 13: Net-(J1-Pin_13) -> 43
- J13 pad 14: Net-(J1-Pin_14) -> 44
- J13 pad 15: Net-(J1-Pin_16) -> 46
- J13 pad 16: Net-(J1-Pin_17) -> 47
- J13 pad 17: Net-(J1-Pin_18) -> 48
- J13 pad 18: Net-(J1-Pin_19) -> 49
- J13 pad 19: Net-(J1-Pin_20) -> 50
- J13 pad 2: Net-(J1-Pin_2) -> 32
- J13 pad 20: Net-(J1-Pin_21) -> 51
- J13 pad 21: Net-(J1-Pin_22) -> 52
- J13 pad 22: Net-(J1-Pin_23) -> 53
- J13 pad 23: Net-(J1-Pin_24) -> 54
- J13 pad 24: Net-(J1-Pin_25) -> 55
- J13 pad 25: Net-(J1-Pin_26) -> 56
- J13 pad 26: Net-(J1-Pin_27) -> 57
- J13 pad 27: Net-(J1-Pin_28) -> 58
- J13 pad 28: Net-(J1-Pin_29) -> 59
- J13 pad 29: Net-(J10-Pin_2) -> 29
- J13 pad 3: Net-(J1-Pin_3) -> 33
- J13 pad 30: Net-(J10-Pin_3) -> 28
- J13 pad 31: Net-(J10-Pin_4) -> 27
- J13 pad 32: Net-(J10-Pin_5) -> 26
- J13 pad 33: Net-(J10-Pin_6) -> 25
- J13 pad 34: Net-(J10-Pin_7) -> 24
- J13 pad 35: Net-(J10-Pin_8) -> 23
- J13 pad 36: Net-(J10-Pin_9) -> 22
- J13 pad 37: Net-(J10-Pin_10) -> 21
- J13 pad 38: Net-(J10-Pin_11) -> 20
- J13 pad 39: Net-(J10-Pin_12) -> 19
- J13 pad 4: Net-(J1-Pin_4) -> 34
- J13 pad 40: Net-(J10-Pin_13) -> 18
- J13 pad 41: Net-(J10-Pin_14) -> 17
- J13 pad 42: Net-(J10-Pin_15) -> 16
- J13 pad 43: Net-(J10-Pin_17) -> 14
- J13 pad 44: Net-(J10-Pin_18) -> 13
- J13 pad 45: Net-(J10-Pin_19) -> 12
- J13 pad 46: Net-(J10-Pin_20) -> 11
- J13 pad 47: Net-(J10-Pin_21) -> 10
- J13 pad 48: Net-(J10-Pin_22) -> 9
- J13 pad 49: Net-(J10-Pin_23) -> 8
- J13 pad 5: Net-(J1-Pin_5) -> 35
- J13 pad 50: Net-(J10-Pin_24) -> 7
- J13 pad 51: Net-(J10-Pin_25) -> 6
- J13 pad 52: Net-(J10-Pin_26) -> 5
- J13 pad 53: Net-(J10-Pin_27) -> 4
- J13 pad 54: Net-(J10-Pin_28) -> 3
- J13 pad 55: Net-(J10-Pin_29) -> 2
- J13 pad 56: Net-(J10-Pin_30) -> 1
- J13 pad 6: Net-(J1-Pin_6) -> 36
- J13 pad 7: Net-(J1-Pin_7) -> 37
- J13 pad 8: Net-(J1-Pin_8) -> 38
- J13 pad 9: Net-(J1-Pin_9) -> 39
- J14 pad 1: Net-(J1-Pin_1) -> 31
- J14 pad 10: Net-(J1-Pin_10) -> 40
- J14 pad 11: Net-(J1-Pin_11) -> 41
- J14 pad 12: Net-(J1-Pin_12) -> 42
- J14 pad 13: Net-(J1-Pin_13) -> 43
- J14 pad 14: Net-(J1-Pin_14) -> 44
- J14 pad 15: Net-(J1-Pin_16) -> 46
- J14 pad 16: Net-(J1-Pin_17) -> 47
- J14 pad 17: Net-(J1-Pin_18) -> 48
- J14 pad 18: Net-(J1-Pin_19) -> 49
- J14 pad 19: Net-(J1-Pin_20) -> 50
- J14 pad 2: Net-(J1-Pin_2) -> 32
- J14 pad 20: Net-(J1-Pin_21) -> 51
- J14 pad 21: Net-(J1-Pin_22) -> 52
- J14 pad 22: Net-(J1-Pin_23) -> 53
- J14 pad 23: Net-(J1-Pin_24) -> 54
- J14 pad 24: Net-(J1-Pin_25) -> 55
- J14 pad 25: Net-(J1-Pin_26) -> 56
- J14 pad 26: Net-(J1-Pin_27) -> 57
- J14 pad 27: Net-(J1-Pin_28) -> 58
- J14 pad 28: Net-(J1-Pin_29) -> 59
- J14 pad 29: Net-(J10-Pin_2) -> 29
- J14 pad 3: Net-(J1-Pin_3) -> 33
- J14 pad 30: Net-(J10-Pin_3) -> 28
- J14 pad 31: Net-(J10-Pin_4) -> 27
- J14 pad 32: Net-(J10-Pin_5) -> 26
- J14 pad 33: Net-(J10-Pin_6) -> 25
- J14 pad 34: Net-(J10-Pin_7) -> 24
- J14 pad 35: Net-(J10-Pin_8) -> 23
- J14 pad 36: Net-(J10-Pin_9) -> 22
- J14 pad 37: Net-(J10-Pin_10) -> 21
- J14 pad 38: Net-(J10-Pin_11) -> 20
- J14 pad 39: Net-(J10-Pin_12) -> 19
- J14 pad 4: Net-(J1-Pin_4) -> 34
- J14 pad 40: Net-(J10-Pin_13) -> 18
- J14 pad 41: Net-(J10-Pin_14) -> 17
- J14 pad 42: Net-(J10-Pin_15) -> 16
- J14 pad 43: Net-(J10-Pin_17) -> 14
- J14 pad 44: Net-(J10-Pin_18) -> 13
- J14 pad 45: Net-(J10-Pin_19) -> 12
- J14 pad 46: Net-(J10-Pin_20) -> 11
- J14 pad 47: Net-(J10-Pin_21) -> 10
- J14 pad 48: Net-(J10-Pin_22) -> 9
- J14 pad 49: Net-(J10-Pin_23) -> 8
- J14 pad 5: Net-(J1-Pin_5) -> 35
- J14 pad 50: Net-(J10-Pin_24) -> 7
- J14 pad 51: Net-(J10-Pin_25) -> 6
- J14 pad 52: Net-(J10-Pin_26) -> 5
- J14 pad 53: Net-(J10-Pin_27) -> 4
- J14 pad 54: Net-(J10-Pin_28) -> 3
- J14 pad 55: Net-(J10-Pin_29) -> 2
- J14 pad 56: Net-(J10-Pin_30) -> 1
- J14 pad 6: Net-(J1-Pin_6) -> 36
- J14 pad 7: Net-(J1-Pin_7) -> 37
- J14 pad 8: Net-(J1-Pin_8) -> 38
- J14 pad 9: Net-(J1-Pin_9) -> 39
- J15 pad 1: Net-(J10-Pin_30) -> 1
- J15 pad 10: Net-(J10-Pin_21) -> 10
- J15 pad 11: Net-(J10-Pin_20) -> 11
- J15 pad 12: Net-(J10-Pin_19) -> 12
- J15 pad 13: Net-(J10-Pin_18) -> 13
- J15 pad 14: Net-(J10-Pin_17) -> 14
- J15 pad 15: Net-(J10-Pin_16) -> 15
- J15 pad 16: Net-(J10-Pin_15) -> 16
- J15 pad 17: Net-(J10-Pin_14) -> 17
- J15 pad 18: Net-(J10-Pin_13) -> 18
- J15 pad 19: Net-(J10-Pin_12) -> 19
- J15 pad 2: Net-(J10-Pin_29) -> 2
- J15 pad 20: Net-(J10-Pin_11) -> 20
- J15 pad 21: Net-(J10-Pin_10) -> 21
- J15 pad 22: Net-(J10-Pin_9) -> 22
- J15 pad 23: Net-(J10-Pin_8) -> 23
- J15 pad 24: Net-(J10-Pin_7) -> 24
- J15 pad 25: Net-(J10-Pin_6) -> 25
- J15 pad 26: Net-(J10-Pin_5) -> 26
- J15 pad 27: Net-(J10-Pin_4) -> 27
- J15 pad 28: Net-(J10-Pin_3) -> 28
- J15 pad 29: Net-(J10-Pin_2) -> 29
- J15 pad 3: Net-(J10-Pin_28) -> 3
- J15 pad 30: Net-(J10-Pin_1) -> 30
- J15 pad 31: Net-(J1-Pin_30) -> 60
- J15 pad 32: Net-(J1-Pin_29) -> 59
- J15 pad 33: Net-(J1-Pin_28) -> 58
- J15 pad 34: Net-(J1-Pin_27) -> 57
- J15 pad 35: Net-(J1-Pin_26) -> 56
- J15 pad 36: Net-(J1-Pin_25) -> 55
- J15 pad 37: Net-(J1-Pin_24) -> 54
- J15 pad 38: Net-(J1-Pin_23) -> 53
- J15 pad 39: Net-(J1-Pin_22) -> 52
- J15 pad 4: Net-(J10-Pin_27) -> 4
- J15 pad 40: Net-(J1-Pin_21) -> 51
- J15 pad 41: Net-(J1-Pin_20) -> 50
- J15 pad 42: Net-(J1-Pin_19) -> 49
- J15 pad 43: Net-(J1-Pin_18) -> 48
- J15 pad 44: Net-(J1-Pin_17) -> 47
- J15 pad 45: Net-(J1-Pin_16) -> 46
- J15 pad 46: Net-(J1-Pin_15) -> 45
- J15 pad 47: Net-(J1-Pin_14) -> 44
- J15 pad 48: Net-(J1-Pin_13) -> 43
- J15 pad 49: Net-(J1-Pin_12) -> 42
- J15 pad 5: Net-(J10-Pin_26) -> 5
- J15 pad 50: Net-(J1-Pin_11) -> 41
- J15 pad 51: Net-(J1-Pin_10) -> 40
- J15 pad 52: Net-(J1-Pin_9) -> 39
- J15 pad 53: Net-(J1-Pin_8) -> 38
- J15 pad 54: Net-(J1-Pin_7) -> 37
- J15 pad 55: Net-(J1-Pin_6) -> 36
- J15 pad 56: Net-(J1-Pin_5) -> 35
- J15 pad 57: Net-(J1-Pin_4) -> 34
- J15 pad 58: Net-(J1-Pin_3) -> 33
- J15 pad 59: Net-(J1-Pin_2) -> 32
- J15 pad 6: Net-(J10-Pin_25) -> 6
- J15 pad 60: Net-(J1-Pin_1) -> 31
- J15 pad 7: Net-(J10-Pin_24) -> 7
- J15 pad 8: Net-(J10-Pin_23) -> 8
- J15 pad 9: Net-(J10-Pin_22) -> 9
- J16 pad 1: Net-(J1-Pin_1) -> 31
- J16 pad 10: Net-(J1-Pin_10) -> 40
- J16 pad 11: Net-(J1-Pin_11) -> 41
- J16 pad 12: Net-(J1-Pin_12) -> 42
- J16 pad 13: Net-(J1-Pin_13) -> 43
- J16 pad 14: Net-(J1-Pin_14) -> 44
- J16 pad 15: Net-(J1-Pin_16) -> 46
- J16 pad 16: Net-(J1-Pin_17) -> 47
- J16 pad 17: Net-(J1-Pin_18) -> 48
- J16 pad 18: Net-(J1-Pin_19) -> 49
- J16 pad 19: Net-(J1-Pin_20) -> 50
- J16 pad 2: Net-(J1-Pin_2) -> 32
- J16 pad 20: Net-(J1-Pin_21) -> 51
- J16 pad 21: Net-(J1-Pin_22) -> 52
- J16 pad 22: Net-(J1-Pin_23) -> 53
- J16 pad 23: Net-(J1-Pin_24) -> 54
- J16 pad 24: Net-(J1-Pin_25) -> 55
- J16 pad 25: Net-(J1-Pin_26) -> 56
- J16 pad 26: Net-(J1-Pin_27) -> 57
- J16 pad 27: Net-(J1-Pin_28) -> 58
- J16 pad 28: Net-(J1-Pin_29) -> 59
- J16 pad 29: Net-(J10-Pin_2) -> 29
- J16 pad 3: Net-(J1-Pin_3) -> 33
- J16 pad 30: Net-(J10-Pin_3) -> 28
- J16 pad 31: Net-(J10-Pin_4) -> 27
- J16 pad 32: Net-(J10-Pin_5) -> 26
- J16 pad 33: Net-(J10-Pin_6) -> 25
- J16 pad 34: Net-(J10-Pin_7) -> 24
- J16 pad 35: Net-(J10-Pin_8) -> 23
- J16 pad 36: Net-(J10-Pin_9) -> 22
- J16 pad 37: Net-(J10-Pin_10) -> 21
- J16 pad 38: Net-(J10-Pin_11) -> 20
- J16 pad 39: Net-(J10-Pin_12) -> 19
- J16 pad 4: Net-(J1-Pin_4) -> 34
- J16 pad 40: Net-(J10-Pin_13) -> 18
- J16 pad 41: Net-(J10-Pin_14) -> 17
- J16 pad 42: Net-(J10-Pin_15) -> 16
- J16 pad 43: Net-(J10-Pin_17) -> 14
- J16 pad 44: Net-(J10-Pin_18) -> 13
- J16 pad 45: Net-(J10-Pin_19) -> 12
- J16 pad 46: Net-(J10-Pin_20) -> 11
- J16 pad 47: Net-(J10-Pin_21) -> 10
- J16 pad 48: Net-(J10-Pin_22) -> 9
- J16 pad 49: Net-(J10-Pin_23) -> 8
- J16 pad 5: Net-(J1-Pin_5) -> 35
- J16 pad 50: Net-(J10-Pin_24) -> 7
- J16 pad 51: Net-(J10-Pin_25) -> 6
- J16 pad 52: Net-(J10-Pin_26) -> 5
- J16 pad 53: Net-(J10-Pin_27) -> 4
- J16 pad 54: Net-(J10-Pin_28) -> 3
- J16 pad 55: Net-(J10-Pin_29) -> 2
- J16 pad 56: Net-(J10-Pin_30) -> 1
- J16 pad 6: Net-(J1-Pin_6) -> 36
- J16 pad 7: Net-(J1-Pin_7) -> 37
- J16 pad 8: Net-(J1-Pin_8) -> 38
- J16 pad 9: Net-(J1-Pin_9) -> 39
- J17 pad 1: Net-(J10-Pin_1) -> 31
- J17 pad 10: Net-(J10-Pin_10) -> 40
- J17 pad 11: Net-(J10-Pin_11) -> 41
- J17 pad 12: Net-(J10-Pin_12) -> 42
- J17 pad 13: Net-(J10-Pin_13) -> 43
- J17 pad 14: Net-(J10-Pin_14) -> 44
- J17 pad 15: Net-(J10-Pin_15) -> 45
- J17 pad 16: Net-(J10-Pin_16) -> 46
- J17 pad 17: Net-(J10-Pin_17) -> 47
- J17 pad 18: Net-(J10-Pin_18) -> 48
- J17 pad 19: Net-(J10-Pin_19) -> 49
- J17 pad 2: Net-(J10-Pin_2) -> 32
- J17 pad 20: Net-(J10-Pin_20) -> 50
- J17 pad 21: Net-(J10-Pin_21) -> 51
- J17 pad 22: Net-(J10-Pin_22) -> 52
- J17 pad 23: Net-(J10-Pin_23) -> 53
- J17 pad 24: Net-(J10-Pin_24) -> 54
- J17 pad 25: Net-(J10-Pin_25) -> 55
- J17 pad 26: Net-(J10-Pin_26) -> 56
- J17 pad 27: Net-(J10-Pin_27) -> 57
- J17 pad 28: Net-(J10-Pin_28) -> 58
- J17 pad 29: Net-(J10-Pin_29) -> 59
- J17 pad 3: Net-(J10-Pin_3) -> 33
- J17 pad 30: Net-(J10-Pin_30) -> 60
- J17 pad 4: Net-(J10-Pin_4) -> 34
- J17 pad 5: Net-(J10-Pin_5) -> 35
- J17 pad 6: Net-(J10-Pin_6) -> 36
- J17 pad 7: Net-(J10-Pin_7) -> 37
- J17 pad 8: Net-(J10-Pin_8) -> 38
- J17 pad 9: Net-(J10-Pin_9) -> 39
- J18 pad 1: Net-(J1-Pin_1) -> 1
- J18 pad 10: Net-(J1-Pin_10) -> 10
- J18 pad 11: Net-(J1-Pin_11) -> 11
- J18 pad 12: Net-(J1-Pin_12) -> 12
- J18 pad 13: Net-(J1-Pin_13) -> 13
- J18 pad 14: Net-(J1-Pin_14) -> 14
- J18 pad 15: Net-(J1-Pin_15) -> 15
- J18 pad 16: Net-(J1-Pin_16) -> 16
- J18 pad 17: Net-(J1-Pin_17) -> 17
- J18 pad 18: Net-(J1-Pin_18) -> 18
- J18 pad 19: Net-(J1-Pin_19) -> 19
- J18 pad 2: Net-(J1-Pin_2) -> 2
- J18 pad 20: Net-(J1-Pin_20) -> 20
- J18 pad 21: Net-(J1-Pin_21) -> 21
- J18 pad 22: Net-(J1-Pin_22) -> 22
- J18 pad 23: Net-(J1-Pin_23) -> 23
- J18 pad 24: Net-(J1-Pin_24) -> 24
- J18 pad 25: Net-(J1-Pin_25) -> 25
- J18 pad 26: Net-(J1-Pin_26) -> 26
- J18 pad 27: Net-(J1-Pin_27) -> 27
- J18 pad 28: Net-(J1-Pin_28) -> 28
- J18 pad 29: Net-(J1-Pin_29) -> 29
- J18 pad 3: Net-(J1-Pin_3) -> 3
- J18 pad 30: Net-(J1-Pin_30) -> 30
- J18 pad 4: Net-(J1-Pin_4) -> 4
- J18 pad 5: Net-(J1-Pin_5) -> 5
- J18 pad 6: Net-(J1-Pin_6) -> 6
- J18 pad 7: Net-(J1-Pin_7) -> 7
- J18 pad 8: Net-(J1-Pin_8) -> 8
- J18 pad 9: Net-(J1-Pin_9) -> 9
- U1 pad 1: Net-(U1A-Pin_1-Pad1) -> 1
- U1 pad 10: Net-(U1A-Pin_10-Pad10) -> 10
- U1 pad 11: Net-(U1A-Pin_11-Pad11) -> 11
- U1 pad 12: Net-(U1A-Pin_12-Pad12) -> 12
- U1 pad 13: Net-(U1A-Pin_13-Pad13) -> 13
- U1 pad 14: Net-(U1A-Pin_14-Pad14) -> 14
- U1 pad 15: Net-(U1A-Pin_15-Pad15) -> 15
- U1 pad 16: Net-(U1A-Pin_16-Pad16) -> 16
- U1 pad 17: Net-(U1A-Pin_17-Pad17) -> 17
- U1 pad 18: Net-(U1A-Pin_18-Pad18) -> 18
- U1 pad 19: Net-(U1A-Pin_19-Pad19) -> 19
- U1 pad 2: Net-(U1A-Pin_2-Pad2) -> 2
- U1 pad 20: Net-(U1A-Pin_20-Pad20) -> 20
- U1 pad 21: Net-(U1A-Pin_21-Pad21) -> 21
- U1 pad 22: Net-(U1A-Pin_22-Pad22) -> 22
- U1 pad 23: Net-(U1A-Pin_23-Pad23) -> 23
- U1 pad 24: Net-(U1A-Pin_24-Pad24) -> 24
- U1 pad 25: Net-(U1A-Pin_25-Pad25) -> 25
- U1 pad 26: Net-(U1A-Pin_26-Pad26) -> 26
- U1 pad 27: Net-(U1A-Pin_27-Pad27) -> 27
- U1 pad 28: Net-(U1A-Pin_28-Pad28) -> 28
- U1 pad 29: Net-(U1A-Pin_29) -> 29
- U1 pad 3: Net-(U1A-Pin_3-Pad3) -> 3
- U1 pad 30: Net-(U1A-Pin_30) -> 30
- U1 pad 31: Net-(U1A-Pin_31) -> 31
- U1 pad 32: Net-(U1A-Pin_0) -> 32
- U1 pad 33: Net-(U1A-Pin_1-Pad33) -> 33
- U1 pad 34: Net-(U1A-Pin_2-Pad34) -> 34
- U1 pad 35: Net-(U1A-Pin_3-Pad35) -> 35
- U1 pad 36: Net-(U1A-Pin_4-Pad36) -> 36
- U1 pad 37: Net-(U1A-Pin_5-Pad37) -> 37
- U1 pad 38: Net-(U1A-Pin_6-Pad38) -> 38
- U1 pad 39: Net-(U1A-Pin_7-Pad39) -> 39
- U1 pad 4: Net-(U1A-Pin_4-Pad4) -> 4
- U1 pad 40: Net-(U1A-Pin_8-Pad40) -> 40
- U1 pad 41: Net-(U1A-Pin_9-Pad41) -> 41
- U1 pad 42: Net-(U1A-Pin_10-Pad42) -> 42
- U1 pad 43: Net-(U1A-Pin_11-Pad43) -> 43
- U1 pad 44: Net-(U1A-Pin_12-Pad44) -> 44
- U1 pad 45: Net-(U1A-Pin_13-Pad45) -> 45
- U1 pad 46: Net-(U1A-Pin_14-Pad46) -> 46
- U1 pad 47: Net-(U1A-Pin_15-Pad47) -> 47
- U1 pad 48: Net-(U1A-Pin_16-Pad48) -> 48
- U1 pad 49: Net-(U1A-Pin_17-Pad49) -> 49
- U1 pad 5: Net-(U1A-Pin_5-Pad5) -> 5
- U1 pad 50: Net-(U1A-Pin_18-Pad50) -> 50
- U1 pad 51: Net-(U1A-Pin_19-Pad51) -> 51
- U1 pad 52: Net-(U1A-Pin_20-Pad52) -> 52
- U1 pad 53: Net-(U1A-Pin_21-Pad53) -> 53
- U1 pad 54: Net-(U1A-Pin_22-Pad54) -> 54
- U1 pad 55: Net-(U1A-Pin_23-Pad55) -> 55
- U1 pad 56: Net-(U1A-Pin_24-Pad56) -> 56
- U1 pad 57: Net-(U1A-Pin_25-Pad57) -> 57
- U1 pad 58: Net-(U1A-Pin_26-Pad58) -> 58
- U1 pad 59: Net-(U1A-Pin_27-Pad59) -> 59
- U1 pad 6: Net-(U1A-Pin_6-Pad6) -> 6
- U1 pad 60: Net-(U1A-Pin_28-Pad60) -> 60
- U1 pad 61: Net-(J1-Pin_1) -> TOP_RAIL_POS
- U1 pad 68: Net-(J8-Pin_1) -> GND
- U1 pad 7: Net-(U1A-Pin_7-Pad7) -> 7
- U1 pad 70: Net-(J10-Pin_1) -> LED_5V
- U1 pad 8: Net-(U1A-Pin_8-Pad8) -> 8
- U1 pad 9: Net-(U1A-Pin_9-Pad9) -> 9
- U3 pad 1: Net-(U1A-Pin_1-Pad1) -> 1
- U3 pad 10: Net-(U1A-Pin_10-Pad10) -> 10
- U3 pad 11: Net-(U1A-Pin_11-Pad11) -> 11
- U3 pad 12: Net-(U1A-Pin_12-Pad12) -> 12
- U3 pad 13: Net-(U1A-Pin_13-Pad13) -> 13
- U3 pad 14: Net-(U1A-Pin_14-Pad14) -> 14
- U3 pad 15: Net-(U1A-Pin_15-Pad15) -> 15
- U3 pad 16: Net-(U1A-Pin_16-Pad16) -> 16
- U3 pad 17: Net-(U1A-Pin_17-Pad17) -> 17
- U3 pad 18: Net-(U1A-Pin_18-Pad18) -> 18
- U3 pad 19: Net-(U1A-Pin_19-Pad19) -> 19
- U3 pad 2: Net-(U1A-Pin_2-Pad2) -> 2
- U3 pad 20: Net-(U1A-Pin_20-Pad20) -> 20
- U3 pad 21: Net-(U1A-Pin_21-Pad21) -> 21
- U3 pad 22: Net-(U1A-Pin_22-Pad22) -> 22
- U3 pad 23: Net-(U1A-Pin_23-Pad23) -> 23
- U3 pad 24: Net-(U1A-Pin_24-Pad24) -> 24
- U3 pad 25: Net-(U1A-Pin_25-Pad25) -> 25
- U3 pad 26: Net-(U1A-Pin_26-Pad26) -> 26
- U3 pad 27: Net-(U1A-Pin_27-Pad27) -> 27
- U3 pad 28: Net-(U1A-Pin_28-Pad28) -> 28
- U3 pad 29: Net-(U1A-Pin_29) -> 29
- U3 pad 3: Net-(U1A-Pin_3-Pad3) -> 3
- U3 pad 30: Net-(U1A-Pin_30) -> 30
- U3 pad 31: Net-(U1A-Pin_31) -> 31
- U3 pad 32: Net-(U1A-Pin_0) -> 32
- U3 pad 33: Net-(U1A-Pin_1-Pad33) -> 33
- U3 pad 34: Net-(U1A-Pin_2-Pad34) -> 34
- U3 pad 35: Net-(U1A-Pin_3-Pad35) -> 35
- U3 pad 36: Net-(U1A-Pin_4-Pad36) -> 36
- U3 pad 37: Net-(U1A-Pin_5-Pad37) -> 37
- U3 pad 38: Net-(U1A-Pin_6-Pad38) -> 38
- U3 pad 39: Net-(U1A-Pin_7-Pad39) -> 39
- U3 pad 4: Net-(U1A-Pin_4-Pad4) -> 4
- U3 pad 40: Net-(U1A-Pin_8-Pad40) -> 40
- U3 pad 41: Net-(U1A-Pin_9-Pad41) -> 41
- U3 pad 42: Net-(U1A-Pin_10-Pad42) -> 42
- U3 pad 43: Net-(U1A-Pin_11-Pad43) -> 43
- U3 pad 44: Net-(U1A-Pin_12-Pad44) -> 44
- U3 pad 45: Net-(U1A-Pin_13-Pad45) -> 45
- U3 pad 46: Net-(U1A-Pin_14-Pad46) -> 46
- U3 pad 47: Net-(U1A-Pin_15-Pad47) -> 47
- U3 pad 48: Net-(U1A-Pin_16-Pad48) -> 48
- U3 pad 49: Net-(U1A-Pin_17-Pad49) -> 49
- U3 pad 5: Net-(U1A-Pin_5-Pad5) -> 5
- U3 pad 50: Net-(U1A-Pin_18-Pad50) -> 50
- U3 pad 51: Net-(U1A-Pin_19-Pad51) -> 51
- U3 pad 52: Net-(U1A-Pin_20-Pad52) -> 52
- U3 pad 53: Net-(U1A-Pin_21-Pad53) -> 53
- U3 pad 54: Net-(U1A-Pin_22-Pad54) -> 54
- U3 pad 55: Net-(U1A-Pin_23-Pad55) -> 55
- U3 pad 56: Net-(U1A-Pin_24-Pad56) -> 56
- U3 pad 57: Net-(U1A-Pin_25-Pad57) -> 57
- U3 pad 58: Net-(U1A-Pin_26-Pad58) -> 58
- U3 pad 59: Net-(U1A-Pin_27-Pad59) -> 59
- U3 pad 6: Net-(U1A-Pin_6-Pad6) -> 6
- U3 pad 60: Net-(U1A-Pin_28-Pad60) -> 60
- U3 pad 61: Net-(J1-Pin_1) -> TOP_RAIL_POS
- U3 pad 68: Net-(J8-Pin_1) -> GND
- U3 pad 7: Net-(U1A-Pin_7-Pad7) -> 7
- U3 pad 70: Net-(J10-Pin_1) -> LED_5V
- U3 pad 8: Net-(U1A-Pin_8-Pad8) -> 8
- U3 pad 9: Net-(U1A-Pin_9-Pad9) -> 9
Routing:
- net 27: track 0.00 -> 225.9 mm, vias 0 -> 6
- net 59: track 0.00 -> 221.0 mm, vias 0 -> 6
- net 26: track 0.00 -> 215.7 mm, vias 0 -> 6
- net 29: track 0.00 -> 214.2 mm, vias 0 -> 7
- net 58: track 0.00 -> 214.0 mm, vias 0 -> 6
- net 57: track 0.00 -> 211.7 mm, vias 0 -> 5
- net 28: track 0.00 -> 207.5 mm, vias 0 -> 7
- net 56: track 0.00 -> 206.3 mm, vias 0 -> 5
- net 25: track 0.00 -> 203.3 mm, vias 0 -> 6
- net 52: track 0.00 -> 201.8 mm, vias 0 -> 5
- net 14: track 0.00 -> 199.7 mm, vias 0 -> 7
- net 13: track 0.00 -> 198.4 mm, vias 0 -> 6
- net 12: track 0.00 -> 194.7 mm, vias 0 -> 6
- net 24: track 0.00 -> 193.4 mm, vias 0 -> 6
- net Net-(J10-Pin_4): track 191.6 -> 0.00 mm, vias 5 -> 0
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Other:
- board size 82.6 x 17.3 mm -> 82.5 x 42.6 mm
- board text added: "1 2 3 4 5 6 7 8 9 10 11 12 13 14 15 16 17 18 19 20 21 22 23 24 25 26 27 28 29 30"
- board text added: "14 13 12 11 10 9 8 7 6 5 4 3 2"
- board text added: "14 13 12 11 10 9 8 7 6 5 4 3 2 1"
- board text added: "16 17 18 19 20 21 22 23 24 25 26 27"
- board text added: "16 17 18 19 20 21 22 23 24 25 26 27 28"
- board text added: "16 17 18 19 20 21 22 23 24 25 26 27 28 29"
- board text added: "17 18 19 20 21 22 23 24 25 26 27"
- board text added: "28"
- board text added: "29"
- board text added: "31 32 33 34 35 36 37 38 39 40 41 42 43 44 45 46 47 48 49 50 51 52 53 54 55 56 57 58 59 60"
- board text added: "31 32 33 34 35 36 37 38 39 41 42 43 44 45"
- board text added: "32 33 34 35 36 37 38 39 41 42 43 44 45"
- board text added: "57 56 55 54 53 52 51 50 49 48 47 46"
- board text added: "58"
- board text added: "58 57 56 55 54 53 52 51 50 49 48 47"
- board text added: "59"
- board text added: "59 58"
- board text removed: "30"
- board text removed: "5V"
- board text removed: "60"
- board text removed: "Data IN"
- board text removed: "GND"
- board text removed: "RP2040"
- board text removed: "WS2812C"
