File: Barnacles/ProtoSMD/ProtoSMD.kicad_pcb (KiCad board)
At the start: 4 copper layers, 174 x 48.3 mm, 33 parts, among them J1 Conn_01x01, J12 Conn_02x03_Top_Bottom, J12 Conn_02x32_Top_Bottom, J13 Conn_02x03_Top_Bottom, J13 Conn_02x32_Top_Bottom, J17 Conn_01x30, J18 Conn_01x30, J2 Conn_01x01, J3 Conn_01x01, J4 Conn_01x01, J5 Conn_01x01, J6 Conn_01x01

Commit message: addProtoSMD
Parts:
- removed the J1 at (224.3, 73.6)
- removed J17: Conn_01x30, JumperlessFootprints:Conn_1x30_breadboard_single
- removed the J2 at (225.8, 73.6)
- removed the J3 at (183.9, 73.6)
- removed the J4 at (182.4, 73.6)
- removed the J5 at (204.1, 73.6)
- removed the REF** at (245.4, 66.5)
- removed the REF** at (162.9, 66.5)
- removed the U1 at (229.5, 80.8)
- removed U2: ~, JumperlessFootprints:Conn_8x30_breadboard
- removed the U3 at (234.6, 30.6)
- added J11: Conn_01x30, JumperlessFootprints:Conn_5x30_breadboard_sin_passives, F.Cu at (113.9, 76.9)
- added J15: Conn_02x08_Counter_Clockwise, JumperlessFootprints:Lines_P1.27_16, F.Cu at (137.4, 56.6)
- added J16: Conn_02x08_Counter_Clockwise, JumperlessFootprints:Lines_P0.65_16, F.Cu at (119.3, 56.6)
- added J19: Conn_02x08_Counter_Clockwise, JumperlessFootprints:Lines_P0.5_16, F.Cu at (99.5, 56.6)
- added J20: Conn_02x06_Counter_Clockwise, JumperlessFootprints:Lines_P0.4_12, F.Cu at (84.4, 56.6)
- added J21: Conn_02x07_Counter_Clockwise, JumperlessFootprints:SOIC14_SOT23-8-6, F.Cu at (93.0, 56.6)
- added J22: Conn_02x03_Counter_Clockwise, Package_TO_SOT_SMD:SOT-223, F.Cu at (79.6, 56.5)
- added J25: Conn_01x03_Pin, Package_TO_SOT_THT:TO-92, F.Cu at (128.5, 56.0)
- added J26: Conn_01x03_Pin, Package_TO_SOT_THT:TO-92, F.Cu at (132.4, 57.3)
- added J27: Conn_02x03_Counter_Clockwise, JumperlessFootprints:LED_6_SMD, F.Cu at (107.6, 56.6)
- added J28: Conn_02x03_Counter_Clockwise, JumperlessFootprints:LED_6_SMD, F.Cu at (115.2, 56.6)
- added J29: Conn_02x08_Counter_Clockwise, Connector_PinHeader_1.27mm:PinHeader_2x08_P1.27mm_Vertical, F.Cu at (151.1, 52.2)
- added J30: Conn_02x10_Counter_Clockwise, JumperlessFootprints:FPC FC05-S20FCT, F.Cu at (148.1, 51.9)
- added J65: Conn_2Rows-13Pins, nixies-us:nixies-us-IN-16, F.Cu at (130.4, 56.6)
- J12: value Conn_02x32_Top_Bottom -> Conn_01x30
- J12: value Conn_02x03_Top_Bottom -> Conn_01x30
- J13: value Conn_02x03_Top_Bottom -> Conn_02x30_Top_Bottom
- J13: value Conn_02x32_Top_Bottom -> Conn_02x30_Top_Bottom
- J18: footprint JumperlessFootprints:Conn_1x30_breadboard_single -> JumperlessFootprints:Conn_5x30_breadboard_sin_passives
- moved J18 91.0 mm to (113.9, 49.0)
- moved REF** 6.33 mm to (155.2, 142.6)
- moved REF** 6.33 mm to (72.7, 142.6)
- moved J6 6.33 mm to (149.4, 155.0)
- moved J1 6.33 mm to (134.1, 81.1)
- moved J12 6.33 mm to (155.2, 97.3)
- moved J2 6.33 mm to (135.7, 81.1)
- moved U1 6.33 mm to (139.3, 88.4)
- moved J1 6.33 mm to (113.9, 99.0)
- moved J3 6.33 mm to (93.7, 81.1)
- moved J4 6.33 mm to (92.2, 81.1)
- moved J5 6.33 mm to (113.9, 81.1)
- moved REF** 6.33 mm to (72.7, 71.5)
- moved J13 6.33 mm to (72.7, 97.2)
- moved REF** 6.33 mm to (155.2, 71.4)
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Connections:
- J1 pad 1: Net-(J1-Pin_1) -> TOP_RAIL_POS
- J2 pad 1: Net-(J2-Pin_1) -> TOP_RAIL_NEG
- J3 pad 1: Net-(J3-Pin_1) -> BOT_RAIL_POS
- J4 pad 1: Net-(J4-Pin_1) -> BOT_RAIL_NEG
- J5 pad 1: Net-(J5-Pin_1) -> PASS
- U1 pad 1: Net-(U1A-Pin_1-Pad1) -> 1
- U1 pad 10: Net-(U1A-Pin_10-Pad10) -> 10
- U1 pad 11: Net-(U1A-Pin_11-Pad11) -> 11
- U1 pad 12: Net-(U1A-Pin_12-Pad12) -> 12
- U1 pad 13: Net-(U1A-Pin_13-Pad13) -> 13
- U1 pad 14: Net-(U1A-Pin_14-Pad14) -> 14
- U1 pad 15: Net-(U1A-Pin_15-Pad15) -> 15
- U1 pad 16: Net-(U1A-Pin_16-Pad16) -> 16
- U1 pad 17: Net-(U1A-Pin_17-Pad17) -> 17
- U1 pad 18: Net-(U1A-Pin_18-Pad18) -> 18
- U1 pad 19: Net-(U1A-Pin_19-Pad19) -> 19
- U1 pad 2: Net-(U1A-Pin_2-Pad2) -> 2
- U1 pad 20: Net-(U1A-Pin_20-Pad20) -> 20
- U1 pad 21: Net-(U1A-Pin_21-Pad21) -> 21
- U1 pad 22: Net-(U1A-Pin_22-Pad22) -> 22
- U1 pad 23: Net-(U1A-Pin_23-Pad23) -> 23
- U1 pad 24: Net-(U1A-Pin_24-Pad24) -> 24
- U1 pad 25: Net-(U1A-Pin_25-Pad25) -> 25
- U1 pad 26: Net-(U1A-Pin_26-Pad26) -> 26
- U1 pad 27: Net-(U1A-Pin_27-Pad27) -> 27
- U1 pad 28: Net-(U1A-Pin_28-Pad28) -> 28
- U1 pad 29: Net-(U1A-Pin_29) -> 29
- U1 pad 3: Net-(U1A-Pin_3-Pad3) -> 3
- U1 pad 30: Net-(U1A-Pin_30) -> 30
- U1 pad 31: Net-(U1A-Pin_31) -> 31
- U1 pad 32: Net-(U1A-Pin_0) -> 32
- U1 pad 33: Net-(U1A-Pin_1-Pad33) -> 33
- U1 pad 34: Net-(U1A-Pin_2-Pad34) -> 34
- U1 pad 35: Net-(U1A-Pin_3-Pad35) -> 35
- U1 pad 36: Net-(U1A-Pin_4-Pad36) -> 36
- U1 pad 37: Net-(U1A-Pin_5-Pad37) -> 37
- U1 pad 38: Net-(U1A-Pin_6-Pad38) -> 38
- U1 pad 39: Net-(U1A-Pin_7-Pad39) -> 39
- U1 pad 4: Net-(U1A-Pin_4-Pad4) -> 4
- U1 pad 40: Net-(U1A-Pin_8-Pad40) -> 40
- U1 pad 41: Net-(U1A-Pin_9-Pad41) -> 41
- U1 pad 42: Net-(U1A-Pin_10-Pad42) -> 42
- U1 pad 43: Net-(U1A-Pin_11-Pad43) -> 43
- U1 pad 44: Net-(U1A-Pin_12-Pad44) -> 44
- U1 pad 45: Net-(U1A-Pin_13-Pad45) -> 45
- U1 pad 46: Net-(U1A-Pin_14-Pad46) -> 46
- U1 pad 47: Net-(U1A-Pin_15-Pad47) -> 47
- U1 pad 48: Net-(U1A-Pin_16-Pad48) -> 48
- U1 pad 49: Net-(U1A-Pin_17-Pad49) -> 49
- U1 pad 5: Net-(U1A-Pin_5-Pad5) -> 5
- U1 pad 50: Net-(U1A-Pin_18-Pad50) -> 50
- U1 pad 51: Net-(U1A-Pin_19-Pad51) -> 51
- U1 pad 52: Net-(U1A-Pin_20-Pad52) -> 52
- U1 pad 53: Net-(U1A-Pin_21-Pad53) -> 53
- U1 pad 54: Net-(U1A-Pin_22-Pad54) -> 54
- U1 pad 55: Net-(U1A-Pin_23-Pad55) -> 55
- U1 pad 56: Net-(U1A-Pin_24-Pad56) -> 56
- U1 pad 57: Net-(U1A-Pin_25-Pad57) -> 57
- U1 pad 58: Net-(U1A-Pin_26-Pad58) -> 58
- U1 pad 59: Net-(U1A-Pin_27-Pad59) -> 59
- U1 pad 6: Net-(U1A-Pin_6-Pad6) -> 6
- U1 pad 60: Net-(U1A-Pin_28-Pad60) -> 60
- U1 pad 61: Net-(J1-Pin_1) -> TOP_RAIL_POS
- U1 pad 62: Net-(J2-Pin_1) -> TOP_RAIL_NEG
- U1 pad 63: Net-(J3-Pin_1) -> BOT_RAIL_POS
- U1 pad 64: Net-(J4-Pin_1) -> BOT_RAIL_NEG
- U1 pad 65: Net-(J5-Pin_1) -> PASS
- U1 pad 66: Net-(J6-Pin_1) -> SENSE_TOP
- U1 pad 67: Net-(J7-Pin_1) -> SENSE_BOTTOM
- U1 pad 68: Net-(J8-Pin_1) -> GND
- U1 pad 69: Net-(J9-Pin_1) -> LED_DAT
- U1 pad 7: Net-(U1A-Pin_7-Pad7) -> 7
- U1 pad 70: Net-(J10-Pin_1) -> LED_5V
- U1 pad 8: Net-(U1A-Pin_8-Pad8) -> 8
- U1 pad 9: Net-(U1A-Pin_9-Pad9) -> 9
- U3 pad 1: Net-(U1A-Pin_1-Pad1) -> 1
- U3 pad 10: Net-(U1A-Pin_10-Pad10) -> 10
- U3 pad 11: Net-(U1A-Pin_11-Pad11) -> 11
- U3 pad 12: Net-(U1A-Pin_12-Pad12) -> 12
- U3 pad 13: Net-(U1A-Pin_13-Pad13) -> 13
- U3 pad 14: Net-(U1A-Pin_14-Pad14) -> 14
- U3 pad 15: Net-(U1A-Pin_15-Pad15) -> 15
- U3 pad 16: Net-(U1A-Pin_16-Pad16) -> 16
- U3 pad 17: Net-(U1A-Pin_17-Pad17) -> 17
- U3 pad 18: Net-(U1A-Pin_18-Pad18) -> 18
- U3 pad 19: Net-(U1A-Pin_19-Pad19) -> 19
- U3 pad 2: Net-(U1A-Pin_2-Pad2) -> 2
- U3 pad 20: Net-(U1A-Pin_20-Pad20) -> 20
- U3 pad 21: Net-(U1A-Pin_21-Pad21) -> 21
- U3 pad 22: Net-(U1A-Pin_22-Pad22) -> 22
- U3 pad 23: Net-(U1A-Pin_23-Pad23) -> 23
- U3 pad 24: Net-(U1A-Pin_24-Pad24) -> 24
- U3 pad 25: Net-(U1A-Pin_25-Pad25) -> 25
- U3 pad 26: Net-(U1A-Pin_26-Pad26) -> 26
- U3 pad 27: Net-(U1A-Pin_27-Pad27) -> 27
- U3 pad 28: Net-(U1A-Pin_28-Pad28) -> 28
- U3 pad 29: Net-(U1A-Pin_29) -> 29
- U3 pad 3: Net-(U1A-Pin_3-Pad3) -> 3
- U3 pad 30: Net-(U1A-Pin_30) -> 30
- U3 pad 31: Net-(U1A-Pin_31) -> 31
- U3 pad 32: Net-(U1A-Pin_0) -> 32
- U3 pad 33: Net-(U1A-Pin_1-Pad33) -> 33
- U3 pad 34: Net-(U1A-Pin_2-Pad34) -> 34
- U3 pad 35: Net-(U1A-Pin_3-Pad35) -> 35
- U3 pad 36: Net-(U1A-Pin_4-Pad36) -> 36
- U3 pad 37: Net-(U1A-Pin_5-Pad37) -> 37
- U3 pad 38: Net-(U1A-Pin_6-Pad38) -> 38
- U3 pad 39: Net-(U1A-Pin_7-Pad39) -> 39
- U3 pad 4: Net-(U1A-Pin_4-Pad4) -> 4
- U3 pad 40: Net-(U1A-Pin_8-Pad40) -> 40
- U3 pad 41: Net-(U1A-Pin_9-Pad41) -> 41
- U3 pad 42: Net-(U1A-Pin_10-Pad42) -> 42
- U3 pad 43: Net-(U1A-Pin_11-Pad43) -> 43
- U3 pad 44: Net-(U1A-Pin_12-Pad44) -> 44
- U3 pad 45: Net-(U1A-Pin_13-Pad45) -> 45
- U3 pad 46: Net-(U1A-Pin_14-Pad46) -> 46
- U3 pad 47: Net-(U1A-Pin_15-Pad47) -> 47
- U3 pad 48: Net-(U1A-Pin_16-Pad48) -> 48
- U3 pad 49: Net-(U1A-Pin_17-Pad49) -> 49
- U3 pad 5: Net-(U1A-Pin_5-Pad5) -> 5
- U3 pad 50: Net-(U1A-Pin_18-Pad50) -> 50
- U3 pad 51: Net-(U1A-Pin_19-Pad51) -> 51
- U3 pad 52: Net-(U1A-Pin_20-Pad52) -> 52
- U3 pad 53: Net-(U1A-Pin_21-Pad53) -> 53
- U3 pad 54: Net-(U1A-Pin_22-Pad54) -> 54
- U3 pad 55: Net-(U1A-Pin_23-Pad55) -> 55
- U3 pad 56: Net-(U1A-Pin_24-Pad56) -> 56
- U3 pad 57: Net-(U1A-Pin_25-Pad57) -> 57
- U3 pad 58: Net-(U1A-Pin_26-Pad58) -> 58
- U3 pad 59: Net-(U1A-Pin_27-Pad59) -> 59
- U3 pad 6: Net-(U1A-Pin_6-Pad6) -> 6
- U3 pad 60: Net-(U1A-Pin_28-Pad60) -> 60
- U3 pad 61: Net-(J1-Pin_1) -> TOP_RAIL_POS
- U3 pad 62: Net-(J2-Pin_1) -> TOP_RAIL_NEG
- U3 pad 63: Net-(J3-Pin_1) -> BOT_RAIL_POS
- U3 pad 64: Net-(J4-Pin_1) -> BOT_RAIL_NEG
- U3 pad 65: Net-(J5-Pin_1) -> PASS
- U3 pad 66: Net-(J6-Pin_1) -> SENSE_TOP
- U3 pad 67: Net-(J7-Pin_1) -> SENSE_BOTTOM
- U3 pad 68: Net-(J8-Pin_1) -> GND
- U3 pad 69: Net-(J9-Pin_1) -> LED_DAT
- U3 pad 7: Net-(U1A-Pin_7-Pad7) -> 7
- U3 pad 70: Net-(J10-Pin_1) -> LED_5V
- U3 pad 8: Net-(U1A-Pin_8-Pad8) -> 8
- U3 pad 9: Net-(U1A-Pin_9-Pad9) -> 9
Routing:
- net (no net): track 1.82 -> 103.7 mm
- net Net-(J1-Pin_1): track 83.5 -> 0.00 mm
- net Net-(J10-Pin_1): track 82.9 -> 0.00 mm
- net SENSE_TOP: track 0.00 -> 82.8 mm
- net Net-(J6-Pin_1): track 82.4 -> 0.00 mm
- net BOT_RAIL_POS: track 0.21 -> 82.5 mm
- net Net-(J3-Pin_1): track 82.2 -> 0.00 mm
- net Net-(J2-Pin_1): track 81.4 -> 0.00 mm
- net Net-(J9-Pin_1): track 81.3 -> 0.00 mm
- net SENSE_BOTTOM: track 0.00 -> 80.9 mm
- net BOT_RAIL_NEG: track 0.15 -> 80.8 mm
- net Net-(J7-Pin_1): track 80.5 -> 0.00 mm
- net Net-(J4-Pin_1): track 80.4 -> 0.00 mm
- net 23: track 21.1 -> 92.9 mm, vias 1 -> 3
- net 51: track 19.5 -> 87.5 mm, vias 1 -> 2
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Other:
- board size 174 x 48.3 mm -> 82.5 x 48.3 mm
- copper layers 4 -> 2
- board text added: "1 2 3 4 5 6"
- board text added: "31 32 33 34 35 36"
- board text removed: "0.4 mm"
- board text removed: "1"
- board text removed: "16"
- board text removed: "16 17 18 19 20 21 22 23 24 25 26 27 28 29"
- board text removed: "28"
- board text removed: "29"
- board text removed: "31"
- board text removed: "46"
- board text removed: "58"
- board text removed: "58 57 56 55 54 53 52 51 50 49 48 47"
- board text removed: "59"
- board text removed: "59 58"
- board text removed: "SOIC/SSOP"
