File: Barnacles/ProtoSMD/ProtoSMD.kicad_pcb (KiCad board)
At the start: 2 copper layers, 82.5 x 48.3 mm, 36 parts, among them J1 Conn_01x01, J11 Conn_01x30, J12 Conn_01x30, J13 Conn_02x30_Top_Bottom, J15 Conn_02x08_Counter_Clockwise, J16 Conn_02x08_Counter_Clockwise, J18 Conn_01x30, J19 Conn_02x08_Counter_Clockwise, J2 Conn_01x01, J20 Conn_02x06_Counter_Clockwise, J21 Conn_02x07_Counter_Clockwise, J22 Conn_02x03_Counter_Clockwise, J25 Conn_01x03_Pin, J26 Conn_01x03_Pin, J27 Conn_02x03_Counter_Clockwise, J28 Conn_02x03_Counter_Clockwise, J29 Conn_02x08_Counter_Clockwise, J3 Conn_01x01, J30 Conn_02x10_Counter_Clockwise, J4 Conn_01x01, J5 Conn_01x01, J6 Conn_01x01, J65 Conn_2Rows-13Pins

Commit message: add wigs
Parts:
- removed the J1 at (-8.61, 84.2)
- removed the J12 at (32.7, 82.5)
- removed the J13 at (-49.9, 82.4)
- removed the J6 at (26.8, 140.2)
- removed the REF** at (-49.9, 127.7)
- removed the REF** at (32.7, 127.7)
Routing:
- net (no net): track 103.7 -> 0.00 mm
- net 58: track 77.8 -> 78.6 mm
- net 39: track 62.7 -> 62.0 mm
- net 42: track 51.9 -> 52.6 mm
- net 56: track 77.7 -> 78.3 mm
- net 29: track 81.4 -> 81.9 mm
- added copper zone on B.Cu, net (none)
Other:
- board text added: "0.4"
- board text added: "0.5"
- board text added: "0.65"
- board text added: "1.27"
- board text added: "Row labels will be wrong if you plug it in with this side up"
- board text removed: "0.5 mm"
- board text removed: "0.65 mm"
- board text removed: "0.8 mm"
- board text removed: "1 2 3 4 5 6"
- board text removed: "1 2 3 4 5 6 7 8 9 10 11 12 13 14 15 16 17 18 19 20 21 22 23 24 25 26 27 28 29 30"
- board text removed: "1.27/0.65mm"
- board text removed: "14 13 12 11 10 9 8 7 6 5 4 3 2"
- board text removed: "14 13 12 11 10 9 8 7 6 5 4 3 2 1"
- board text removed: "16 17 18 19 20 21 22 23 24 25 26 27"
- board text removed: "16 17 18 19 20 21 22 23 24 25 26 27 28"
- board text removed: "17 18 19 20 21 22 23 24 25 26 27"
- board text removed: "31 32 33 34 35 36"
- board text removed: "31 32 33 34 35 36 37 38 39 40 41 42 43 44 45 46 47 48 49 50 51 52 53 54 55 56 57 58 59 60"
- board text removed: "31 32 33 34 35 36 37 38 39 41 42 43 44 45"
- board text removed: "32 33 34 35 36 37 38 39 41 42 43 44 45"
- board text removed: "57 56 55 54 53 52 51 50 49 48 47 46"
- board text removed: "QFN/QFP"
