File: Barnacles/ProtoSMD/ProtoSMD.kicad_sch (KiCad schematic)
At the start: 33 parts, among them J1 Conn_01x01, J10 Conn_01x01, J11 Conn_01x30, J12 Conn_01x30, J13 Conn_02x30_Top_Bottom, J14 Conn_02x30_Top_Bottom, J15 Conn_02x08_Counter_Clockwise, J16 Conn_02x08_Counter_Clockwise, J17 Conn_01x30, J18 Conn_01x30, J19 Conn_02x08_Counter_Clockwise, J2 Conn_01x01, J20 Conn_02x06_Counter_Clockwise, J21 Conn_02x07_Counter_Clockwise, J22 Conn_02x03_Counter_Clockwise, J23 Conn_01x01, J25 Conn_01x03_Pin, J26 Conn_01x03_Pin, J27 Conn_02x03_Counter_Clockwise, J28 Conn_02x03_Counter_Clockwise, J29 Conn_02x08_Counter_Clockwise, J3 Conn_01x01, J30 Conn_02x10_Counter_Clockwise, J4 Conn_01x01, J5 Conn_01x01, J6 Conn_01x01, J65 Conn_2Rows-13Pins, J7 Conn_01x01, J8 Conn_01x01, J9 Conn_01x01

Commit message: ugh
Parts:
- D1: symbol Device:LED -> JumperlessSymbols:LED
- J11, J12, J17, J18: symbol Connector_Generic:Conn_01x30 -> JumperlessSymbols:Conn_01x30
- J13, J14: symbol Connector_Generic:Conn_02x30_Top_Bottom -> JumperlessSymbols:Conn_02x30_Top_Bottom
- J15, J16, J19, J29: symbol Connector_Generic:Conn_02x08_Counter_Clockwise -> JumperlessSymbols:Conn_02x08_Counter_Clockwise
- J20: symbol Connector_Generic:Conn_02x06_Counter_Clockwise -> JumperlessSymbols:Conn_02x06_Counter_Clockwise
- J21: symbol Connector_Generic:Conn_02x07_Counter_Clockwise -> JumperlessSymbols:Conn_02x07_Counter_Clockwise
- J22: symbol Connector_Generic:Conn_02x03_Counter_Clockwise -> JumperlessSymbols:Conn_02x03_Counter_Clockwise
- J23: symbol Connector_Generic:Conn_01x01 -> JumperlessSymbols:Conn_01x01
- J25, J26: symbol Connector:Conn_01x03_Pin -> JumperlessSymbols:Conn_01x03_Pin
- J27, J28: symbol Connector_Generic:Conn_02x03_Counter_Clockwise -> JumperlessSymbols:Conn_02x03_Counter_Clockwise_1
- J30: symbol Connector_Generic:Conn_02x10_Counter_Clockwise -> JumperlessSymbols:Conn_02x10_Counter_Clockwise
- J65: symbol Connector_Generic:Conn_02x07_Counter_Clockwise -> JumperlessSymbols:Conn_02x07_Counter_Clockwise_1
- U1, U3: value ~ -> (none); symbol JumperlessSymbols:Breadboard_BBunits -> JumperlessSymbols:Breadboard_BBunits_1
