File: Barnacles/protoSMDfootprintField/protoSMDfootprintField.kicad_sch (KiCad schematic)
At the start: 33 parts, among them J1 Conn_01x01, J10 Conn_01x01, J11 Conn_01x30, J12 Conn_01x30, J13 Conn_02x30_Top_Bottom, J14 Conn_02x30_Top_Bottom, J15 Conn_02x08_Counter_Clockwise, J16 Conn_02x08_Counter_Clockwise, J17 Conn_01x30, J18 Conn_01x30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

Commit message: addProtoSMD
Connections:
- net SENSE_BOTTOM: no longer U3.67 (PadSense_Bottom)
Changed lines of the file:
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@@
 	(global_label "SENSE_BOTTOM"
 		(shape input)
-		(at 113.03 354.33 180)
+		(at 161.29 217.17 180)
 		(fields_autoplaced yes)
 		(effects
@@
 		)
 		(property "Intersheetrefs" "${INTERSHEET_REFS}"
-			(at 95.7121 354.33 0)
+			(at 143.9721 217.17 0)
 			(effects
 				(font
