File: Barnacles/Proto/Proto.kicad_sch (KiCad schematic)
At the start: 13 parts, among them J1 Conn_01x01, J10 Conn_01x01, J2 Conn_01x01, J3 Conn_01x01, J4 Conn_01x01, J5 Conn_01x01, J6 Conn_01x01, J7 Conn_01x01, J8 Conn_01x01, J9 Conn_01x01

Commit message: add wigs
Parts:
- U1, U2, U3: value ~ -> (none)
